Commit message: commit urdf model with joints configured incomplete, servo and legs not implemented

File: src/simulations/ws/src/quadruped/urdf/quadruped.urdf (robot description, URDF)
Before this commit: robot myfirst, 6 links, 4 joints
Links:
- added link leg_bottom_pivot_plate_1; visual mesh filename=package://quadruped/meshes/leg_bottom_pivot_plate.stl
- added link leg_bottom_pivot_plate_2; visual mesh filename=package://quadruped/meshes/leg_bottom_pivot_plate.stl
- added link leg_bottom_pivot_plate_3; visual mesh filename=package://quadruped/meshes/leg_bottom_pivot_plate.stl
- added link leg_bottom_pivot_plate_4; visual mesh filename=package://quadruped/meshes/leg_bottom_pivot_plate.stl
Joints:
- added joint base_top_joint: type fixed, parent base_link, child body_top_plate, origin xyz=0 0.875 0
- added joint leg_bottom_pivot_plate_1: type revolute, parent base_link, child leg_bottom_pivot_plate_1, origin xyz=1.7806 0 1.7806, axis 1.7806 0 1.7806, limit lower=-1.571 upper=1.571 effort=100 velocity=100
- added joint leg_bottom_pivot_plate_2: type revolute, parent base_link, child leg_bottom_pivot_plate_2, origin xyz=-1.7806 0 1.7806, axis 1.7806 0 1.7806, limit lower=-1.571 upper=1.571 effort=100 velocity=100
- added joint leg_bottom_pivot_plate_3: type revolute, parent base_link, child leg_bottom_pivot_plate_3, origin xyz=-1.7806 0 -1.7806, axis -1.7806 0 -1.7806, limit lower=-1.571 upper=1.571 effort=100 velocity=100
- added joint leg_bottom_pivot_plate_4: type revolute, parent base_link, child leg_bottom_pivot_plate_4, origin xyz=1.7806 0 -1.7806, axis 1.7806 0 -1.7806, limit lower=-1.571 upper=1.571 effort=100 velocity=100
- joint base_body_spacer_1: origin (none) -> xyz=0 0 1.700
- joint base_body_spacer_2: origin (none) -> xyz=1.700 0 0
- joint base_body_spacer_3: origin (none) -> xyz=-1.700 0 0
- joint base_body_spacer_4: origin (none) -> xyz=0 0 -1.700

Commit message: commit servo needs scaling and origin also needs to be fixed

File: src/simulations/ws/src/quadruped/urdf/quadruped.urdf (robot description, URDF)
Before this commit: robot myfirst, 10 links, 9 joints
Links:
- added link servo_1; visual mesh filename=package://quadruped/meshes/servo.stl
Joints:
- added joint base_servo_1: type fixed, parent base_link, child servo_1, origin xyz=0 0 0

Commit message: commit quadruped body done, legs remaining

File: src/simulations/ws/src/quadruped/urdf/quadruped.urdf (robot description, URDF)
Before this commit: robot myfirst, 11 links, 10 joints
Links:
- added link retainer_1; visual mesh filename=package://quadruped/meshes/leg_servo_retainer.stl
- added link servo_2; visual mesh filename=package://quadruped/meshes/servo_motor.stl scale=0.1 0.1 0.1
- added link servo_3; visual mesh filename=package://quadruped/meshes/servo_motor.stl scale=0.1 0.1 0.1
- added link servo_4; visual mesh filename=package://quadruped/meshes/servo_motor.stl scale=0.1 0.1 0.1
- link servo_1: geometry visual mesh filename=package://quadruped/meshes/servo_motor.stl scale=0.1 0.1 0.1
Joints:
- removed joint base_servo_1
- added joint servo_retainer_1: type fixed, parent servo_1, child retainer_1
- added joint servo_top_1: type fixed, parent body_top_plate, child servo_1, origin xyz=1.7806 0.375 1.7806
- added joint servo_top_2: type fixed, parent body_top_plate, child servo_2, origin xyz=-1.7806 0.375 1.7806
- added joint servo_top_3: type fixed, parent body_top_plate, child servo_3, origin xyz=-1.7806 0.375 -1.7806
- added joint servo_top_4: type fixed, parent body_top_plate, child servo_4, origin xyz=1.7806 0.375 -1.7806

Commit message: commit hip joint complete need to fix a slight positioning issue

File: src/simulations/ws/src/quadruped/urdf/quadruped.urdf (robot description, URDF)
Before this commit: robot myfirst, 15 links, 14 joints
Links:
- added link leg_parallel_plate_1; visual mesh filename=package://quadruped/meshes/leg_parallel_plate.stl
- added link leg_parallel_plate_2; visual mesh filename=package://quadruped/meshes/leg_parallel_plate.stl
- added link leg_parallel_plate_3; visual mesh filename=package://quadruped/meshes/leg_parallel_plate.stl
- added link leg_parallel_plate_4; visual mesh filename=package://quadruped/meshes/leg_parallel_plate.stl
- added link leg_top_plate_1; visual mesh filename=package://quadruped/meshes/leg_top_plate.stl
- added link leg_top_plate_2; visual mesh filename=package://quadruped/meshes/leg_top_plate.stl
- added link leg_top_plate_3; visual mesh filename=package://quadruped/meshes/leg_top_plate.stl
- added link leg_top_plate_4; visual mesh filename=package://quadruped/meshes/leg_top_plate.stl
Joints:
- added joint leg_parallel_plate_top_plate_1: type fixed, parent leg_top_plate_1, child leg_parallel_plate_1, origin xyz=0.8096 -0.839 0.5168
- added joint leg_parallel_plate_top_plate_2: type fixed, parent leg_top_plate_2, child leg_parallel_plate_2, origin xyz=-0.5168 -0.839 0.8096
- added joint leg_parallel_plate_top_plate_3: type fixed, parent leg_top_plate_3, child leg_parallel_plate_3, origin xyz=-0.8096 -0.839 -0.5168
- added joint leg_parallel_plate_top_plate_4: type fixed, parent leg_top_plate_4, child leg_parallel_plate_4, origin xyz=0.5168 -0.839 -0.8096
- added joint servo_leg_top_plate_1: type revolute, parent servo_1, child leg_top_plate_1, origin xyz=0 0.303 0, axis 0 2.5184 0, limit lower=-1.571 upper=1.571 effort=100 velocity=100
- added joint servo_leg_top_plate_2: type revolute, parent servo_2, child leg_top_plate_2, origin xyz=0 0.303 0, axis 0 2.5184 0, limit lower=-1.571 upper=1.571 effort=100 velocity=100
- added joint servo_leg_top_plate_3: type revolute, parent servo_3, child leg_top_plate_3, origin xyz=0 0.303 0, axis 0 2.5184 0, limit lower=-1.571 upper=1.571 effort=100 velocity=100
- added joint servo_leg_top_plate_4: type revolute, parent servo_4, child leg_top_plate_4, origin xyz=0 0.303 0, axis 0 2.5184 0, limit lower=-1.571 upper=1.571 effort=100 velocity=100
- joint leg_bottom_pivot_plate_1: axis 1.7806 0 1.7806 -> (none); limit lower=-1.571 upper=1.571 effort=100 velocity=100 -> (none); origin xyz=1.7806 0 1.7806 -> xyz=0 -1.563 0; parent base_link -> leg_top_plate_1; type revolute -> fixed
- joint leg_bottom_pivot_plate_2: axis 1.7806 0 1.7806 -> (none); limit lower=-1.571 upper=1.571 effort=100 velocity=100 -> (none); origin xyz=-1.7806 0 1.7806 -> xyz=0 -1.563 0; parent base_link -> leg_top_plate_2; type revolute -> fixed
- joint leg_bottom_pivot_plate_3: axis -1.7806 0 -1.7806 -> (none); limit lower=-1.571 upper=1.571 effort=100 velocity=100 -> (none); origin xyz=-1.7806 0 -1.7806 -> xyz=0 -1.563 0; parent base_link -> leg_top_plate_3; type revolute -> fixed
- joint leg_bottom_pivot_plate_4: axis 1.7806 0 -1.7806 -> (none); limit lower=-1.571 upper=1.571 effort=100 velocity=100 -> (none); origin xyz=1.7806 0 -1.7806 -> xyz=0 -1.563 0; parent base_link -> leg_top_plate_4; type revolute -> fixed

Commit message: commit sync

File: src/simulations/ws/src/quadruped/urdf/quadruped.urdf (robot description, URDF)
Before this commit: robot myfirst, 23 links, 22 joints
Links:
- added link leg_servo_mount_1; visual mesh filename=package://quadruped/meshes/leg_servo_mount.stl
Joints:
- added joint leg_servo_mount_top_plate_1: type fixed, parent leg_top_plate_1, child leg_servo_mount_1, origin xyz=0.5168 -0.839 0.8096
- joint servo_leg_top_plate_1: limit lower=-1.571 upper=1.571 effort=100 velocity=100 -> lower=-1.57079 upper=1.57079 effort=100 velocity=100
- joint servo_leg_top_plate_2: limit lower=-1.571 upper=1.571 effort=100 velocity=100 -> lower=-1.57079 upper=1.57079 effort=100 velocity=100
- joint servo_leg_top_plate_3: limit lower=-1.571 upper=1.571 effort=100 velocity=100 -> lower=-1.57079 upper=1.57079 effort=100 velocity=100
- joint servo_leg_top_plate_4: limit lower=-1.571 upper=1.571 effort=100 velocity=100 -> lower=-1.57079 upper=1.57079 effort=100 velocity=100
