Commit message: commit fixed bouncing problem
Former-commit-id: 6567057fccd1340d6a635c7678fdcf8bded2fa80

File: src/simulations/ws/src/quadruped/urdf/quadruped_model.xacro (robot description, xacro)
@@ -7,4 +7,6 @@
     </plugin>
   </gazebo>
+  <xacro:property name="damping_value" value="10" />
+  <xacro:property name="friction_value" value="0.5" />
   <xacro:property name="scaling_factor" value="2.2" />
   <!--height:z width:y width:x -->
@@ -35,6 +37,6 @@
   <xacro:property name="leg3_joint_high" value="${pi*2.0/18.0}" />
   <xacro:property name="leg_tip_mass" value="${(scaling_factor**3)*0.02}" />
-  <xacro:property name="servo_vel" value="4.0" />
-  <xacro:property name="servo_effort_limit" value="50.0" />
+  <xacro:property name="servo_vel" value="10.0" />
+  <xacro:property name="servo_effort_limit" value="100.0" />
   <!-- Import Rviz colors -->
   <xacro:include filename="$(find quadruped)/urdf/materials.xacro" />
@@ -84,5 +86,5 @@
     <parent link="dummy_link"/>
     <child link="base_link"/>
-    <origin xyz="0 0 0" rpy="0 0 0"/>
+    <origin xyz="0 0 ${leg1_height}" rpy="0 0 0"/>
   </joint>
   <gazebo reference="base_link">
@@ -113,4 +115,5 @@
     <child link="imu_link"/>
     <origin xyz="0 0 ${(body_height/2.0)+(imu_size/2.0)}" rpy="0 0 0"/>
+    <dynamics damping="${damping_value}" friction="${friction_value}" />
   </joint>
   <gazebo reference="imu_link">
@@ -160,4 +163,5 @@
       <child link="${prefix}_${suffix}_leg_tip"/>
       <origin xyz="0 ${-reflect_right*leg1_width/2.0} ${-leg1_height-leg1_depth*1.41/4.0}" rpy="0 0 0"/>
+      <dynamics damping="${damping_value}" friction="${friction_value}" />
     </joint>
     <gazebo reference="${prefix}_${suffix}_leg_tip">
@@ -214,5 +218,5 @@
       <origin xyz="${leg2_depth*cos(pi-leg2_init_pitch)} 0 ${leg2_depth*sin(pi-leg2_init_pitch)}" rpy="0 ${-pi+leg2_init_pitch} 0"/>
       <limit lower="${leg1_joint_low}" upper="${leg1_joint_high}" effort="${servo_effort_limit}" velocity="${servo_vel}"/>
-      <dynamics friction="0.0" />
+      <dynamics damping="${damping_value}" friction="${friction_value}" />
     </joint>
     <gazebo reference="${prefix}_${suffix}_leg1">
@@ -245,5 +249,5 @@
       <origin xyz="${leg3_depth/2.0} ${reflect_right*leg3_width/2.0} 0" />
       <limit lower="${leg2_joint_low}" upper="${leg2_joint_high}" effort="${servo_effort_limit}" velocity="${servo_vel}"/>
-      <dynamics friction="0.0" />
+      <dynamics damping="${damping_value}" friction="${friction_value}" />
     </joint>
     <gazebo reference="${prefix}_${suffix}_leg2">
@@ -276,5 +280,5 @@
       <origin xyz="${reflect_right*body_width/2.0} ${reflect_front*body_width/2.0} 0" rpy="0 0 ${reflect_front*pi/2.0 - reflect_front*reflect_right*pi/4.0}"/>
       <limit lower="${leg3_joint_low}" upper="${leg3_joint_high}" effort="${servo_effort_limit}" velocity="${servo_vel}"/>
-      <dynamics friction="0.0" />
+      <dynamics damping="${damping_value}" friction="${friction_value}" />
     </joint>
     <gazebo reference="${prefix}_${suffix}_leg3">
@@ -307,9 +311,9 @@
     <transmission name="tran${num}">
       <joint name="${front_back}_${right_left}_${leg}_joint">
-        <hardwareInterface>hardware_interface/EffortJointInterface</hardwareInterface>
+        <hardwareInterface>hardware_interface/PositionJointInterface</hardwareInterface>
       </joint>
       <type>transmission_interface/SimpleTransmission</type>
       <actuator name="servo${num}">
-        <hardwareInterface>hardware_interface/EffortJointInterface</hardwareInterface>
+        <hardwareInterface>hardware_interface/PositionJointInterface</hardwareInterface>
         <mechanicalReduction>1</mechanicalReduction>
       </actuator>

Commit message: commit functional contact sensor
Former-commit-id: b585630cd8add9249bfcc19a028f4e829c198efa

File: src/simulations/ws/src/quadruped/urdf/quadruped_model.xacro (robot description, xacro)
@@ -151,5 +151,5 @@
         <material name="black"/>
       </visual>
-      <collision>
+      <collision name="${prefix}_${suffix}_leg_tip">
         <origin xyz="0 0 0" rpy="0 0 0" />
         <geometry>
@@ -167,5 +167,5 @@
     <gazebo reference="${prefix}_${suffix}_leg_tip">
       <minDepth>0.0002</minDepth>
-      <collision name="${prefix}_${suffix}_leg_tip_collision_1">
+      <collision name="${prefix}_${suffix}_leg_tip_collision">
         <geometry>
           <sphere>
@@ -188,4 +188,18 @@
         </surface>
       </collision>
+      <sensor name="${prefix}_${suffix}_leg_tip_contact_sensor" type="contact">
+        <plugin name="gazebo_ros_bumper_controller" filename="libgazebo_ros_bumper.so">
+          <robotNamespace>/quadruped</robotNamespace>
+          <bumperTopicName>${prefix}_${suffix}_leg_tip_contact_sensor</bumperTopicName>
+          <frameName>${prefix}_${suffix}_leg_tip</frameName>
+          <alwayson>true</alwayson>
+          <updaterate>100</updaterate>
+        </plugin>
+        <always_on>true</always_on>
+        <update_rate>100</update_rate>
+        <contact>
+          <collision>${prefix}_${suffix}_leg_tip_collision</collision>
+        </contact>
+      </sensor>
       <material>Gazebo/Black</material>
     </gazebo>

Commit message: commit moveit planner setup done need to fix an error with planner configuratio
Former-commit-id: e6fcbc381ef3aa97e122a5ea1578595536405e6a

File: src/simulations/ws/src/quadruped/urdf/quadruped_model.xacro (robot description, xacro)
@@ -54,4 +54,7 @@
     </inertial>
   </xacro:macro>
+  <!-- Dummmy -->
+  <link name="dummy">
+  </link>
   <!-- Quadruped -->
   <link name="dummy_link">
@@ -69,4 +72,8 @@
     </gazebo>
   </link>
+  <joint name="dummy_joint" type="fixed">
+     <parent link="dummy"/>
+     <child link="dummy_link"/>
+   </joint>
   <link name="base_link">
     <visual>

Commit message: commit force torque sensor functional stability reward calculation done energy reward computation to be set up
Former-commit-id: 28c05f83b7aebb3d5633ced2a276b7b63d7e6eb0

File: src/simulations/ws/src/quadruped/urdf/quadruped_model.xacro (robot description, xacro)
@@ -7,6 +7,6 @@
     </plugin>
   </gazebo>
-  <xacro:property name="damping_value" value="10" />
-  <xacro:property name="friction_value" value="0.5" />
+  <xacro:property name="damping_value" value="0.1" />
+  <xacro:property name="friction_value" value="0.05" />
   <xacro:property name="scaling_factor" value="2.2" />
   <!--height:z width:y width:x -->
@@ -37,5 +37,5 @@
   <xacro:property name="leg3_joint_high" value="${pi*2.0/18.0}" />
   <xacro:property name="leg_tip_mass" value="${(scaling_factor**3)*0.02}" />
-  <xacro:property name="servo_vel" value="10.0" />
+  <xacro:property name="servo_vel" value="100.0" />
   <xacro:property name="servo_effort_limit" value="100.0" />
   <!-- Import Rviz colors -->
@@ -96,6 +96,7 @@
   </joint>
   <gazebo reference="base_link">
-    <mu1>100000.0</mu1>
-    <mu2>100000.0</mu2>
+    <gravity>true</gravity>
+    <mu1>${friction_value}</mu1>
+    <mu2>${friction_value}</mu2>
     <material>Gazebo/Black</material>
   </gazebo>
@@ -173,4 +174,5 @@
     </joint>
     <gazebo reference="${prefix}_${suffix}_leg_tip">
+      <gravity>true</gravity>
       <minDepth>0.0002</minDepth>
       <collision name="${prefix}_${suffix}_leg_tip_collision">
@@ -183,9 +185,9 @@
           <friction>
             <ode>
-              <mu>100000.0</mu>
-              <mu2>100000.0</mu2>
+              <mu>${friction_value}</mu>
+              <mu2>${friction_value}</mu2>
             </ode>
             <torsional>
-              <coefficient>1000000</coefficient>
+              <coefficient>${friction_value}</coefficient>
               <use_patch_radius>true</use_patch_radius>
               <surface_radius>${leg1_depth/2.0}</surface_radius>
@@ -242,7 +244,28 @@
     </joint>
     <gazebo reference="${prefix}_${suffix}_leg1">
-      <mu1>100000.0</mu1>
-      <mu2>100000.0</mu2>
+      <gravity>true</gravity>
+      <mu1>${friction_value}</mu1>
+      <mu2>${friction_value}</mu2>
       <material>Gazebo/White</material>
+    </gazebo>
+    <gazebo reference="${prefix}_${suffix}_leg2_joint">
+      <provideFeedback>true</provideFeedback>
+      <sensor name="${prefix}_${suffix}_leg1_joint_force_torque" type="force_torque">
+        <always_on>true</always_on>
+        <update_rate>100.0</update_rate>
+      </sensor>
+    </gazebo>
+    <gazebo>
+      <plugin name="ft_sensor" filename="libgazebo_ros_ft_sensor.so">
+        <robotNamespace>/quadruped</robotNamespace>
+        <topicName>${prefix}_${suffix}_leg1_joint_force_torque</topicName>
+        <jointName>${prefix}_${suffix}_leg1_joint</jointName>
+        <noise>
+          <type>gaussian</type>
+          <mean>0.0</mean>
+          <stddev>0.003</stddev>
+          <!-- change this to simulate noise -->
+        </noise>
+      </plugin>
     </gazebo>
   </xacro:macro>
@@ -273,7 +296,28 @@
     </joint>
     <gazebo reference="${prefix}_${suffix}_leg2">
-      <mu1>100000.0</mu1>
-      <mu2>100000.0</mu2>
+      <gravity>true</gravity>
+      <mu1>${friction_value}</mu1>
+      <mu2>${friction_value}</mu2>
       <material>Gazebo/Black</material>
+    </gazebo>
+    <gazebo reference="${prefix}_${suffix}_leg2_joint">
+      <provideFeedback>true</provideFeedback>
+      <sensor name="${prefix}_${suffix}_leg1_joint_force_torque" type="force_torque">
+        <always_on>true</always_on>
+        <update_rate>100.0</update_rate>
+      </sensor>
+    </gazebo>
+    <gazebo>
+      <plugin name="ft_sensor" filename="libgazebo_ros_ft_sensor.so">
+        <robotNamespace>/quadruped</robotNamespace>
+        <topicName>${prefix}_${suffix}_leg2_joint_force_torque</topicName>
+        <jointName>${prefix}_${suffix}_leg2_joint</jointName>
+        <noise>
+          <type>gaussian</type>
+          <mean>0.0</mean>
+          <stddev>0.003</stddev>
+          <!-- change this to simulate noise -->
+        </noise>
+      </plugin>
     </gazebo>
   </xacro:macro>
@@ -304,6 +348,7 @@
     </joint>
     <gazebo reference="${prefix}_${suffix}_leg3">
-      <mu1>100000.0</mu1>
-      <mu2>100000.0</mu2>
+      <gravity>true</gravity>
+      <mu1>${friction_value}</mu1>
+      <mu2>${friction_value}</mu2>
       <material>Gazebo/White</material>
     </gazebo>

Commit message: commit transform error fixed need to debug reward
Former-commit-id: d608efbe7620cc987c4ac936713089d7904103ee

File: src/simulations/ws/src/quadruped/urdf/quadruped_model.xacro (robot description, xacro)
@@ -54,7 +54,4 @@
     </inertial>
   </xacro:macro>
-  <!-- Dummmy -->
-  <link name="dummy">
-  </link>
   <!-- Quadruped -->
   <link name="dummy_link">
@@ -72,8 +69,4 @@
     </gazebo>
   </link>
-  <joint name="dummy_joint" type="fixed">
-     <parent link="dummy"/>
-     <child link="dummy_link"/>
-   </joint>
   <link name="base_link">
     <visual>
@@ -201,5 +194,5 @@
           <robotNamespace>/quadruped</robotNamespace>
           <bumperTopicName>${prefix}_${suffix}_leg_tip_contact_sensor</bumperTopicName>
-          <frameName>world</frameName>
+          <frameName>dummy_link</frameName>
           <alwayson>true</alwayson>
           <updaterate>100</updaterate>

Commit message: commit gait test for appropriate pretraining input data
Former-commit-id: 7b45010dcab8b0a5d2a395b9c9936d75d55b28f9

File: src/simulations/ws/src/quadruped/urdf/quadruped_model.xacro (robot description, xacro)
@@ -37,6 +37,6 @@
   <xacro:property name="leg3_joint_high" value="${pi*2.0/18.0}" />
   <xacro:property name="leg_tip_mass" value="${(scaling_factor**3)*0.02}" />
-  <xacro:property name="servo_vel" value="100.0" />
-  <xacro:property name="servo_effort_limit" value="100.0" />
+  <xacro:property name="servo_vel" value="9" />
+  <xacro:property name="servo_effort_limit" value="10" />
   <!-- Import Rviz colors -->
   <xacro:include filename="$(find quadruped)/urdf/materials.xacro" />

Commit message: commit modifications for correction of jerks
Former-commit-id: 38ee58674cfaf5601fee61af8533887c7d67555d

File: src/simulations/ws/src/quadruped/urdf/quadruped_model.xacro (robot description, xacro)
@@ -38,5 +38,5 @@
   <xacro:property name="leg_tip_mass" value="${(scaling_factor**3)*0.02}" />
   <xacro:property name="servo_vel" value="9" />
-  <xacro:property name="servo_effort_limit" value="10" />
+  <xacro:property name="servo_effort_limit" value="100" />
   <!-- Import Rviz colors -->
   <xacro:include filename="$(find quadruped)/urdf/materials.xacro" />
@@ -54,4 +54,7 @@
     </inertial>
   </xacro:macro>
+  <!-- Dummmy -->
+  <link name="dummy">
+  </link>
   <!-- Quadruped -->
   <link name="dummy_link">
@@ -69,4 +72,8 @@
     </gazebo>
   </link>
+  <joint name="dummy_joint" type="fixed">
+     <parent link="dummy"/>
+     <child link="dummy_link"/>
+   </joint>
   <link name="base_link">
     <visual>

Commit message: commit new data for pretraining
Former-commit-id: 519c298c65c1ad46abccde74802b40bb4289a7c8

File: src/simulations/ws/src/quadruped/urdf/quadruped_model.xacro (robot description, xacro)
@@ -21,12 +21,12 @@
   <xacro:property name="leg1_depth" value="${scaling_factor*0.015}" />
   <xacro:property name="leg1_mass" value="${(scaling_factor**3)*0.8}" />
-  <xacro:property name="leg1_joint_low" value="${-pi*2.0/18.0}" />
-  <xacro:property name="leg1_joint_high" value="${pi*2.0/18.0}" />
+  <xacro:property name="leg1_joint_low" value="${-pi/3.0}" />
+  <xacro:property name="leg1_joint_high" value="${pi*3.0}" />
   <xacro:property name="leg2_height" value="${scaling_factor*0.025}" />
   <xacro:property name="leg2_width" value="${scaling_factor*0.01}" />
   <xacro:property name="leg2_depth" value="${scaling_factor*0.1}" />
   <xacro:property name="leg2_mass" value="${(scaling_factor**3)*0.05}" />
-  <xacro:property name="leg2_joint_low" value="${-pi*2.0/18.0}" />
-  <xacro:property name="leg2_joint_high" value="${pi*2.0/18.0}" />
+  <xacro:property name="leg2_joint_low" value="${-pi/3.0}" />
+  <xacro:property name="leg2_joint_high" value="${pi/3.0}" />
   <xacro:property name="leg2_init_pitch" value="${pi*16.0/18.0}" />
   <xacro:property name="leg3_height" value="${scaling_factor*0.052}" />
@@ -34,6 +34,6 @@
   <xacro:property name="leg3_depth" value="${scaling_factor*0.015}" />
   <xacro:property name="leg3_mass" value="${(scaling_factor**3)*0.1}" />
-  <xacro:property name="leg3_joint_low" value="${-pi*2.0/18.0}" />
-  <xacro:property name="leg3_joint_high" value="${pi*2.0/18.0}" />
+  <xacro:property name="leg3_joint_low" value="${-pi/3.0}" />
+  <xacro:property name="leg3_joint_high" value="${pi/3.0}" />
   <xacro:property name="leg_tip_mass" value="${(scaling_factor**3)*0.02}" />
   <xacro:property name="servo_vel" value="9" />
