Commit message: commit sync

File: src/simulations/ws/src/Base_link_description/urdf/Base_link.xacro (robot description, xacro)
@@ -124,4 +124,424 @@
   </collision>
 </link>
+<link name="servo_motor_v1_1">
+  <inertial>
+    <origin rpy="0 0 0" xyz="-0.0013508261710446674 0.006780947696453059 0.0013508250495978952"/>
+    <mass value="0.0004848665871049835"/>
+    <inertia ixx="0.0" ixy="0.0" ixz="0.0" iyy="0.0" iyz="-0.0" izz="0.0"/>
+  </inertial>
+  <visual>
+    <origin rpy="0 0 0" xyz="-0.017806 0.00555 0.017806"/>
+    <geometry>
+      <mesh filename="package://Base_link_description/meshes/servo_motor_v1_1.stl" scale="0.001 0.001 0.001"/>
+    </geometry>
+    <material name="silver"/>
+  </visual>
+  <collision>
+    <origin rpy="0 0 0" xyz="-0.017806 0.00555 0.017806"/>
+    <geometry>
+      <mesh filename="package://Base_link_description/meshes/servo_motor_v1_1.stl" scale="0.001 0.001 0.001"/>
+    </geometry>
+  </collision>
+</link>
+<link name="servo_motor_v1_2">
+  <inertial>
+    <origin rpy="0 0 0" xyz="-0.0013508262416907883 0.006780947696453066 0.034261175021048224"/>
+    <mass value="0.0004848665871049835"/>
+    <inertia ixx="0.0" ixy="0.0" ixz="-0.0" iyy="0.0" iyz="0.0" izz="0.0"/>
+  </inertial>
+  <visual>
+    <origin rpy="0 0 0" xyz="-0.017806 0.00555 0.017806"/>
+    <geometry>
+      <mesh filename="package://Base_link_description/meshes/servo_motor_v1_2.stl" scale="0.001 0.001 0.001"/>
+    </geometry>
+    <material name="silver"/>
+  </visual>
+  <collision>
+    <origin rpy="0 0 0" xyz="-0.017806 0.00555 0.017806"/>
+    <geometry>
+      <mesh filename="package://Base_link_description/meshes/servo_motor_v1_2.stl" scale="0.001 0.001 0.001"/>
+    </geometry>
+  </collision>
+</link>
+<link name="servo_motor_v1_3">
+  <inertial>
+    <origin rpy="0 0 0" xyz="-0.03426118356885484 0.006780947696453063 0.034212932907539614"/>
+    <mass value="0.0004848665871049835"/>
+    <inertia ixx="0.0" ixy="-0.0" ixz="0.0" iyy="0.0" iyz="0.0" izz="0.0"/>
+  </inertial>
+  <visual>
+    <origin rpy="0 0 0" xyz="-0.017806 0.00555 0.017806"/>
+    <geometry>
+      <mesh filename="package://Base_link_description/meshes/servo_motor_v1_3.stl" scale="0.001 0.001 0.001"/>
+    </geometry>
+    <material name="silver"/>
+  </visual>
+  <collision>
+    <origin rpy="0 0 0" xyz="-0.017806 0.00555 0.017806"/>
+    <geometry>
+      <mesh filename="package://Base_link_description/meshes/servo_motor_v1_3.stl" scale="0.001 0.001 0.001"/>
+    </geometry>
+  </collision>
+</link>
+<link name="servo_motor_v1_4">
+  <inertial>
+    <origin rpy="0 0 0" xyz="-0.034261183498208725 0.006780947696453061 0.001351940764028104"/>
+    <mass value="0.0004848665871049835"/>
+    <inertia ixx="0.0" ixy="-0.0" ixz="-0.0" iyy="0.0" iyz="-0.0" izz="0.0"/>
+  </inertial>
+  <visual>
+    <origin rpy="0 0 0" xyz="-0.017806 0.00555 0.017806"/>
+    <geometry>
+      <mesh filename="package://Base_link_description/meshes/servo_motor_v1_4.stl" scale="0.001 0.001 0.001"/>
+    </geometry>
+    <material name="silver"/>
+  </visual>
+  <collision>
+    <origin rpy="0 0 0" xyz="-0.017806 0.00555 0.017806"/>
+    <geometry>
+      <mesh filename="package://Base_link_description/meshes/servo_motor_v1_4.stl" scale="0.001 0.001 0.001"/>
+    </geometry>
+  </collision>
+</link>
+<link name="leg_servo_retainer_v1_1">
+  <inertial>
+    <origin rpy="0 0 0" xyz="-7.358861605038722e-05 -0.0006249999403953553 7.439445171635722e-05"/>
+    <mass value="0.0007120198480863978"/>
+    <inertia ixx="0.0" ixy="0.0" ixz="0.0" iyy="0.0" iyz="-0.0" izz="0.0"/>
+  </inertial>
+  <visual>
+    <origin rpy="0 0 0" xyz="-0.016321 0.00127 0.016323"/>
+    <geometry>
+      <mesh filename="package://Base_link_description/meshes/leg_servo_retainer_v1_1.stl" scale="0.001 0.001 0.001"/>
+    </geometry>
+    <material name="silver"/>
+  </visual>
+  <collision>
+    <origin rpy="0 0 0" xyz="-0.016321 0.00127 0.016323"/>
+    <geometry>
+      <mesh filename="package://Base_link_description/meshes/leg_servo_retainer_v1_1.stl" scale="0.001 0.001 0.001"/>
+    </geometry>
+  </collision>
+</link>
+<link name="leg_servo_retainer_v1_2">
+  <inertial>
+    <origin rpy="0 0 0" xyz="-7.409009750477397e-05 -0.0006249999403953553 0.032576253306189185"/>
+    <mass value="0.0007120198480863978"/>
+    <inertia ixx="0.0" ixy="0.0" ixz="-0.0" iyy="0.0" iyz="0.0" izz="0.0"/>
+  </inertial>
+  <visual>
+    <origin rpy="0 0 0" xyz="-0.016321 0.00127 0.016323"/>
+    <geometry>
+      <mesh filename="package://Base_link_description/meshes/leg_servo_retainer_v1_2.stl" scale="0.001 0.001 0.001"/>
+    </geometry>
+    <material name="silver"/>
+  </visual>
+  <collision>
+    <origin rpy="0 0 0" xyz="-0.016321 0.00127 0.016323"/>
+    <geometry>
+      <mesh filename="package://Base_link_description/meshes/leg_servo_retainer_v1_2.stl" scale="0.001 0.001 0.001"/>
+    </geometry>
+  </collision>
+</link>
+<link name="leg_servo_retainer_v1_3">
+  <inertial>
+    <origin rpy="0 0 0" xyz="-0.032575948951977615 -0.0006249999403953564 0.03257575182473469"/>
+    <mass value="0.0007120198480863978"/>
+    <inertia ixx="0.0" ixy="0.0" ixz="0.0" iyy="0.0" iyz="-0.0" izz="0.0"/>
+  </inertial>
+  <visual>
+    <origin rpy="0 0 0" xyz="-0.016321 0.00127 0.016323"/>
+    <geometry>
+      <mesh filename="package://Base_link_description/meshes/leg_servo_retainer_v1_3.stl" scale="0.001 0.001 0.001"/>
+    </geometry>
+    <material name="silver"/>
+  </visual>
+  <collision>
+    <origin rpy="0 0 0" xyz="-0.016321 0.00127 0.016323"/>
+    <geometry>
+      <mesh filename="package://Base_link_description/meshes/leg_servo_retainer_v1_3.stl" scale="0.001 0.001 0.001"/>
+    </geometry>
+  </collision>
+</link>
+<link name="leg_servo_retainer_v1_4">
+  <inertial>
+    <origin rpy="0 0 0" xyz="-0.03255044747052323 -0.0006249999403953551 9.889297026197119e-05"/>
+    <mass value="0.0007120198480863978"/>
+    <inertia ixx="0.0" ixy="0.0" ixz="-0.0" iyy="0.0" iyz="-0.0" izz="0.0"/>
+  </inertial>
+  <visual>
+    <origin rpy="0 0 0" xyz="-0.016321 0.00127 0.016323"/>
+    <geometry>
+      <mesh filename="package://Base_link_description/meshes/leg_servo_retainer_v1_4.stl" scale="0.001 0.001 0.001"/>
+    </geometry>
+    <material name="silver"/>
+  </visual>
+  <collision>
+    <origin rpy="0 0 0" xyz="-0.016321 0.00127 0.016323"/>
+    <geometry>
+      <mesh filename="package://Base_link_description/meshes/leg_servo_retainer_v1_4.stl" scale="0.001 0.001 0.001"/>
+    </geometry>
+  </collision>
+</link>
+<link name="leg_top_pivot_plate_v1_1">
+  <inertial>
+    <origin rpy="0 0 0" xyz="0.004176127215360273 0.0006250000596046473 -0.004148158293409882"/>
+    <mass value="0.0012497785111649892"/>
+    <inertia ixx="0.0" ixy="0.0" ixz="0.0" iyy="0.0" iyz="0.0" izz="0.0"/>
+  </inertial>
+  <visual>
+    <origin rpy="0 0 0" xyz="-0.017806 0.00555 0.017806"/>
+    <geometry>
+      <mesh filename="package://Base_link_description/meshes/leg_top_pivot_plate_v1_1.stl" scale="0.001 0.001 0.001"/>
+    </geometry>
+    <material name="silver"/>
+  </visual>
+  <collision>
+    <origin rpy="0 0 0" xyz="-0.017806 0.00555 0.017806"/>
+    <geometry>
+      <mesh filename="package://Base_link_description/meshes/leg_top_pivot_plate_v1_1.stl" scale="0.001 0.001 0.001"/>
+    </geometry>
+  </collision>
+</link>
+<link name="leg_top_pivot_plate_v1_2">
+  <inertial>
+    <origin rpy="0 0 0" xyz="0.004148157101316982 0.0006250000596046568 0.03978812840745315"/>
+    <mass value="0.0012497785111649892"/>
+    <inertia ixx="0.0" ixy="0.0" ixz="-0.0" iyy="0.0" iyz="0.0" izz="0.0"/>
+  </inertial>
+  <visual>
+    <origin rpy="0 0 0" xyz="-0.017806 0.00555 0.017806"/>
+    <geometry>
+      <mesh filename="package://Base_link_description/meshes/leg_top_pivot_plate_v1_2.stl" scale="0.001 0.001 0.001"/>
+    </geometry>
+    <material name="silver"/>
+  </visual>
+  <collision>
+    <origin rpy="0 0 0" xyz="-0.017806 0.00555 0.017806"/>
+    <geometry>
+      <mesh filename="package://Base_link_description/meshes/leg_top_pivot_plate_v1_2.stl" scale="0.001 0.001 0.001"/>
+    </geometry>
+  </collision>
+</link>
+<link name="leg_top_pivot_plate_v1_3">
+  <inertial>
+    <origin rpy="0 0 0" xyz="-0.039788136955259776 0.0006250000596046508 0.0397119162505474"/>
+    <mass value="0.0012497785111649892"/>
+    <inertia ixx="0.0" ixy="-0.0" ixz="0.0" iyy="0.0" iyz="0.0" izz="0.0"/>
+  </inertial>
+  <visual>
+    <origin rpy="0 0 0" xyz="-0.017806 0.00555 0.017806"/>
+    <geometry>
+      <mesh filename="package://Base_link_description/meshes/leg_top_pivot_plate_v1_3.stl" scale="0.001 0.001 0.001"/>
+    </geometry>
+    <material name="silver"/>
+  </visual>
+  <collision>
+    <origin rpy="0 0 0" xyz="-0.017806 0.00555 0.017806"/>
+    <geometry>
+      <mesh filename="package://Base_link_description/meshes/leg_top_pivot_plate_v1_3.stl" scale="0.001 0.001 0.001"/>
+    </geometry>
+  </collision>
+</link>
+<link name="leg_top_pivot_plate_v1_4">
+  <inertial>
+    <origin rpy="0 0 0" xyz="-0.039760166841216506 0.0006250000596046508 -0.004175012622376836"/>
+    <mass value="0.0012497785111649892"/>
+    <inertia ixx="0.0" ixy="-0.0" ixz="-0.0" iyy="0.0" iyz="-0.0" izz="0.0"/>
+  </inertial>
+  <visual>
+    <origin rpy="0 0 0" xyz="-0.017806 0.00555 0.017806"/>
+    <geometry>
+      <mesh filename="package://Base_link_description/meshes/leg_top_pivot_plate_v1_4.stl" scale="0.001 0.001 0.001"/>
+    </geometry>
+    <material name="silver"/>
+  </visual>
+  <collision>
+    <origin rpy="0 0 0" xyz="-0.017806 0.00555 0.017806"/>
+    <geometry>
+      <mesh filename="package://Base_link_description/meshes/leg_top_pivot_plate_v1_4.stl" scale="0.001 0.001 0.001"/>
+    </geometry>
+  </collision>
+</link>
+<link name="leg_servo_mount_v1_1">
+  <inertial>
+    <origin rpy="0 0 0" xyz="0.00251985940472043 0.004113778478571477 -0.002520105113429757"/>
+    <mass value="0.001144548758330191"/>
+    <inertia ixx="0.0" ixy="-0.0" ixz="0.0" iyy="0.0" iyz="0.0" izz="0.0"/>
+  </inertial>
+  <visual>
+    <origin rpy="0 0 0" xyz="-0.022859 0.00105 0.026465"/>
+    <geometry>
+      <mesh filename="package://Base_link_description/meshes/leg_servo_mount_v1_1.stl" scale="0.001 0.001 0.001"/>
+    </geometry>
+    <material name="silver"/>
+  </visual>
+  <collision>
+    <origin rpy="0 0 0" xyz="-0.022859 0.00105 0.026465"/>
+    <geometry>
+      <mesh filename="package://Base_link_description/meshes/leg_servo_mount_v1_1.stl" scale="0.001 0.001 0.001"/>
+    </geometry>
+  </collision>
+</link>
+<link name="leg_servo_mount_v1_2">
+  <inertial>
+    <origin rpy="0 0 0" xyz="0.006126103921336862 0.004113778478571479 0.051843860596813285"/>
+    <mass value="0.001144548758330191"/>
+    <inertia ixx="0.0" ixy="-0.0" ixz="-0.0" iyy="0.0" iyz="-0.0" izz="0.0"/>
+  </inertial>
+  <visual>
+    <origin rpy="0 0 0" xyz="-0.022859 0.00105 0.026465"/>
+    <geometry>
+      <mesh filename="package://Base_link_description/meshes/leg_servo_mount_v1_2.stl" scale="0.001 0.001 0.001"/>
+    </geometry>
+    <material name="silver"/>
+  </visual>
+  <collision>
+    <origin rpy="0 0 0" xyz="-0.022859 0.00105 0.026465"/>
+    <geometry>
+      <mesh filename="package://Base_link_description/meshes/leg_servo_mount_v1_2.stl" scale="0.001 0.001 0.001"/>
+    </geometry>
+  </collision>
+</link>
+<link name="leg_servo_mount_v1_3">
+  <inertial>
+    <origin rpy="0 0 0" xyz="-0.051844113661236396 0.00411377847857148 0.0010872551882629977"/>
+    <mass value="0.001144548758330191"/>
+    <inertia ixx="0.0" ixy="0.0" ixz="-0.0" iyy="0.0" iyz="0.0" izz="0.0"/>
+  </inertial>
+  <visual>
+    <origin rpy="0 0 0" xyz="-0.022859 0.00105 0.026465"/>
+    <geometry>
+      <mesh filename="package://Base_link_description/meshes/leg_servo_mount_v1_3.stl" scale="0.001 0.001 0.001"/>
+    </geometry>
+    <material name="silver"/>
+  </visual>
+  <collision>
+    <origin rpy="0 0 0" xyz="-0.022859 0.00105 0.026465"/>
+    <geometry>
+      <mesh filename="package://Base_link_description/meshes/leg_servo_mount_v1_3.stl" scale="0.001 0.001 0.001"/>
+    </geometry>
+  </collision>
+</link>
+<link name="leg_servo_mount_v1_4">
+  <inertial>
+    <origin rpy="0 0 0" xyz="-0.04823786914461993 0.004113778478571477 0.05540186307056726"/>
+    <mass value="0.001144548758330191"/>
+    <inertia ixx="0.0" ixy="0.0" ixz="0.0" iyy="0.0" iyz="-0.0" izz="0.0"/>
+  </inertial>
+  <visual>
+    <origin rpy="0 0 0" xyz="-0.022859 0.00105 0.026465"/>
+    <geometry>
+      <mesh filename="package://Base_link_description/meshes/leg_servo_mount_v1_4.stl" scale="0.001 0.001 0.001"/>
+    </geometry>
+    <material name="silver"/>
+  </visual>
+  <collision>
+    <origin rpy="0 0 0" xyz="-0.022859 0.00105 0.026465"/>
+    <geometry>
+      <mesh filename="package://Base_link_description/meshes/leg_servo_mount_v1_4.stl" scale="0.001 0.001 0.001"/>
+    </geometry>
+  </collision>
+</link>
+<link name="leg_parallel_plate_v1_1">
+  <inertial>
+    <origin rpy="0 0 0" xyz="0.00031741714756083547 0.003050233586176742 -0.0003169963388769473"/>
+    <mass value="0.000869495656702597"/>
+    <inertia ixx="0.0" ixy="0.0" ixz="0.0" iyy="0.0" iyz="-0.0" izz="0.0"/>
+  </inertial>
+  <visual>
+    <origin rpy="0 0 0" xyz="-0.026786 0.00105 0.023859"/>
+    <geometry>
+      <mesh filename="package://Base_link_description/meshes/leg_parallel_plate_v1_1.stl" scale="0.001 0.001 0.001"/>
+    </geometry>
+    <material name="silver"/>
+  </visual>
+  <collision>
+    <origin rpy="0 0 0" xyz="-0.026786 0.00105 0.023859"/>
+    <geometry>
+      <mesh filename="package://Base_link_description/meshes/leg_parallel_plate_v1_1.stl" scale="0.001 0.001 0.001"/>
+    </geometry>
+  </collision>
+</link>
+<link name="leg_parallel_plate_v1_2">
+  <inertial>
+    <origin rpy="0 0 0" xyz="-0.0026100048532159345 0.0030502335861767515 0.05096241833965374"/>
+    <mass value="0.000869495656702597"/>
+    <inertia ixx="0.0" ixy="0.0" ixz="-0.0" iyy="0.0" iyz="0.0" izz="0.0"/>
+  </inertial>
+  <visual>
+    <origin rpy="0 0 0" xyz="-0.026786 0.00105 0.023859"/>
+    <geometry>
+      <mesh filename="package://Base_link_description/meshes/leg_parallel_plate_v1_2.stl" scale="0.001 0.001 0.001"/>
+    </geometry>
+    <material name="silver"/>
+  </visual>
+  <collision>
+    <origin rpy="0 0 0" xyz="-0.026786 0.00105 0.023859"/>
+    <geometry>
+      <mesh filename="package://Base_link_description/meshes/leg_parallel_plate_v1_2.stl" scale="0.001 0.001 0.001"/>
+    </geometry>
+  </collision>
+</link>
+<link name="leg_parallel_plate_v1_3">
+  <inertial>
+    <origin rpy="0 0 0" xyz="-0.05096200488668359 0.0030502335861767454 -0.0032433025545774118"/>
+    <mass value="0.000869495656702597"/>
+    <inertia ixx="0.0" ixy="-0.0" ixz="-0.0" iyy="0.0" iyz="-0.0" izz="0.0"/>
+  </inertial>
+  <visual>
+    <origin rpy="0 0 0" xyz="-0.026786 0.00105 0.023859"/>
+    <geometry>
+      <mesh filename="package://Base_link_description/meshes/leg_parallel_plate_v1_3.stl" scale="0.001 0.001 0.001"/>
+    </geometry>
+    <material name="silver"/>
+  </visual>
+  <collision>
+    <origin rpy="0 0 0" xyz="-0.026786 0.00105 0.023859"/>
+    <geometry>
+      <mesh filename="package://Base_link_description/meshes/leg_parallel_plate_v1_3.stl" scale="0.001 0.001 0.001"/>
+    </geometry>
+  </collision>
+</link>
+<link name="leg_parallel_plate_v1_4">
+  <inertial>
+    <origin rpy="0 0 0" xyz="-0.053889426887460366 0.0030502335861767446 0.04798675429601447"/>
+    <mass value="0.000869495656702597"/>
+    <inertia ixx="0.0" ixy="-0.0" ixz="0.0" iyy="0.0" iyz="0.0" izz="0.0"/>
+  </inertial>
+  <visual>
+    <origin rpy="0 0 0" xyz="-0.026786 0.00105 0.023859"/>
+    <geometry>
+      <mesh filename="package://Base_link_description/meshes/leg_parallel_plate_v1_4.stl" scale="0.001 0.001 0.001"/>
+    </geometry>
+    <material name="silver"/>
+  </visual>
+  <collision>
+    <origin rpy="0 0 0" xyz="-0.026786 0.00105 0.023859"/>
+    <geometry>
+      <mesh filename="package://Base_link_description/meshes/leg_parallel_plate_v1_4.stl" scale="0.001 0.001 0.001"/>
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