Commit message: commit removing redundancies in urdf

File: src/simulations/ws/src/quadruped_urdf_description/urdf/quadruped_urdf.xacro (robot description, xacro)
@@ -724,24 +724,4 @@
   </collision>
 </link>
-<link name="leg_parallel_plate_v1_1">
-  <inertial>
-    <origin rpy="0 0 0" xyz="-0.002842085555363149 0.0019600908093042393 -0.003474661877473836"/>
-    <mass value="0.000869495656702597"/>
-    <inertia ixx="0.0" ixy="0.0" ixz="-0.0" iyy="0.0" iyz="0.0" izz="0.0"/>
-  </inertial>
-  <visual>
-    <origin rpy="0 0 0" xyz="-0.027013 0.02844 -0.010983"/>
-    <geometry>
-      <mesh filename="package://quadruped_urdf_description/meshes/leg_parallel_plate_v1_1.stl" scale="0.001 0.001 0.001"/>
-    </geometry>
-    <material name="silver"/>
-  </visual>
-  <collision>
-    <origin rpy="0 0 0" xyz="-0.027013 0.02844 -0.010983"/>
-    <geometry>
-      <mesh filename="package://quadruped_urdf_description/meshes/leg_parallel_plate_v1_1.stl" scale="0.001 0.001 0.001"/>
-    </geometry>
-  </collision>
-</link>
 <link name="leg_rev_v1_1">
   <inertial>
@@ -761,24 +741,4 @@
     <geometry>
       <mesh filename="package://quadruped_urdf_description/meshes/leg_rev_v1_1.stl" scale="0.001 0.001 0.001"/>
-    </geometry>
-  </collision>
-</link>
-<link name="leg_parallel_linkage_v1_1">
-  <inertial>
-    <origin rpy="0 0 0" xyz="-0.003092236328059928 0.0039785038803480804 4.063869700579245e-06"/>
-    <mass value="0.00046200899599845404"/>
-    <inertia ixx="0.0" ixy="0.0" ixz="0.0" iyy="0.0" iyz="-0.0" izz="0.0"/>
-  </inertial>
-  <visual>
-    <origin rpy="0 0 0" xyz="-0.034082 0.035514 -0.010975"/>
-    <geometry>
-      <mesh filename="package://quadruped_urdf_description/meshes/leg_parallel_linkage_v1_1.stl" scale="0.001 0.001 0.001"/>
-    </geometry>
-    <material name="silver"/>
-  </visual>
-  <collision>
-    <origin rpy="0 0 0" xyz="-0.034082 0.035514 -0.010975"/>
-    <geometry>
-      <mesh filename="package://quadruped_urdf_description/meshes/leg_parallel_linkage_v1_1.stl" scale="0.001 0.001 0.001"/>
     </geometry>
   </collision>
@@ -844,44 +804,4 @@
   </collision>
 </link>
-<link name="leg_rev_v1_2">
-  <inertial>
-    <origin rpy="0 0 0" xyz="0.0006852236923735391 -0.00015762169912957036 -0.009769137547065949"/>
-    <mass value="0.001572468577271628"/>
-    <inertia ixx="0.0" ixy="-0.0" ixz="0.0" iyy="0.0" iyz="0.0" izz="0.0"/>
-  </inertial>
-  <visual>
-    <origin rpy="0 0 0" xyz="-0.03646 -0.034334 -0.01123"/>
-    <geometry>
-      <mesh filename="package://quadruped_urdf_description/meshes/leg_rev_v1_2.stl" scale="0.001 0.001 0.001"/>
-    </geometry>
-    <material name="silver"/>
-  </visual>
-  <collision>
-    <origin rpy="0 0 0" xyz="-0.03646 -0.034334 -0.01123"/>
-    <geometry>
-      <mesh filename="package://quadruped_urdf_description/meshes/leg_rev_v1_2.stl" scale="0.001 0.001 0.001"/>
-    </geometry>
-  </collision>
-</link>
-<link name="leg_parallel_plate_v1_2">
-  <inertial>
-    <origin rpy="0 0 0" xyz="-0.0020174799661103367 -0.0028010460511558727 -0.003475778338663464"/>
-    <mass value="0.000869495656702597"/>
-    <inertia ixx="0.0" ixy="-0.0" ixz="-0.0" iyy="0.0" iyz="-0.0" izz="0.0"/>
-  </inertial>
-  <visual>
-    <origin rpy="0 0 0" xyz="-0.029248 -0.027411 -0.010991"/>
-    <geometry>
-      <mesh filename="package://quadruped_urdf_description/meshes/leg_parallel_plate_v1_2.stl" scale="0.001 0.001 0.001"/>
-    </geometry>
-    <material name="silver"/>
-  </visual>
-  <collision>
-    <origin rpy="0 0 0" xyz="-0.029248 -0.027411 -0.010991"/>
-    <geometry>
-      <mesh filename="package://quadruped_urdf_description/meshes/leg_parallel_plate_v1_2.stl" scale="0.001 0.001 0.001"/>
-    </geometry>
-  </collision>
-</link>
 <link name="leg_servo_arm_v1_3">
   <inertial>
@@ -944,44 +864,4 @@
   </collision>
 </link>
-<link name="leg_parallel_linkage_v1_3">
-  <inertial>
-    <origin rpy="0 0 0" xyz="0.0030914923582355154 -0.003978066455700653 -6.215259610374731e-05"/>
-    <mass value="0.00046200899599845404"/>
-    <inertia ixx="0.0" ixy="0.0" ixz="0.0" iyy="0.0" iyz="-0.0" izz="0.0"/>
-  </inertial>
-  <visual>
-    <origin rpy="0 0 0" xyz="0.034083 -0.036716 -0.011123"/>
-    <geometry>
-      <mesh filename="package://quadruped_urdf_description/meshes/leg_parallel_linkage_v1_3.stl" scale="0.001 0.001 0.001"/>
-    </geometry>
-    <material name="silver"/>
-  </visual>
-  <collision>
-    <origin rpy="0 0 0" xyz="0.034083 -0.036716 -0.011123"/>
-    <geometry>
-      <mesh filename="package://quadruped_urdf_description/meshes/leg_parallel_linkage_v1_3.stl" scale="0.001 0.001 0.001"/>
-    </geometry>
-  </collision>
-</link>
-<link name="leg_parallel_plate_v1_3">
-  <inertial>
-    <origin rpy="0 0 0" xyz="0.0028410387917938915 -0.0019594370611173313 -0.003475970717607765"/>
-    <mass value="0.000869495656702597"/>
-    <inertia ixx="0.0" ixy="0.0" ixz="0.0" iyy="0.0" iyz="-0.0" izz="0.0"/>
-  </inertial>
-  <visual>
-    <origin rpy="0 0 0" xyz="0.027015 -0.029643 -0.010999"/>
-    <geometry>
-      <mesh filename="package://quadruped_urdf_description/meshes/leg_parallel_plate_v1_3.stl" scale="0.001 0.001 0.001"/>
-    </geometry>
-    <material name="silver"/>
-  </visual>
-  <collision>
-    <origin rpy="0 0 0" xyz="0.027015 -0.029643 -0.010999"/>
-    <geometry>
-      <mesh filename="package://quadruped_urdf_description/meshes/leg_parallel_plate_v1_3.stl" scale="0.001 0.001 0.001"/>
-    </geometry>
-  </collision>
-</link>
 <link name="leg_servo_arm_v1_4">
   <inertial>
@@ -1041,44 +921,4 @@
     <geometry>
       <mesh filename="package://quadruped_urdf_description/meshes/leg_rev_v1_4.stl" scale="0.001 0.001 0.001"/>
-    </geometry>
-  </collision>
-</link>
-<link name="leg_parallel_linkage_v1_4">
-  <inertial>
-    <origin rpy="0 0 0" xyz="0.0039770161146753386 0.0030932763955820383 8.69419066081012e-08"/>
-    <mass value="0.00046200899599845404"/>
-    <inertia ixx="0.0" ixy="-0.0" ixz="-0.0" iyy="0.0" iyz="0.0" izz="0.0"/>
-  </inertial>
-  <visual>
-    <origin rpy="0 0 0" xyz="0.036134 0.033463 -0.010991"/>
-    <geometry>
-      <mesh filename="package://quadruped_urdf_description/meshes/leg_parallel_linkage_v1_4.stl" scale="0.001 0.001 0.001"/>
-    </geometry>
-    <material name="silver"/>
-  </visual>
-  <collision>
-    <origin rpy="0 0 0" xyz="0.036134 0.033463 -0.010991"/>
-    <geometry>
-      <mesh filename="package://quadruped_urdf_description/meshes/leg_parallel_linkage_v1_4.stl" scale="0.001 0.001 0.001"/>
-    </geometry>
-  </collision>
-</link>
-<link name="leg_parallel_plate_v1_4">
-  <inertial>
-    <origin rpy="0 0 0" xyz="0.0019580207184070574 0.0028430440340579573 -0.0034748931301506105"/>
-    <mass value="0.000869495656702597"/>
-    <inertia ixx="0.0" ixy="-0.0" ixz="0.0" iyy="0.0" iyz="0.0" izz="0.0"/>
-  </inertial>
-  <visual>
-    <origin rpy="0 0 0" xyz="0.029063 0.026392 -0.010991"/>
-    <geometry>
-      <mesh filename="package://quadruped_urdf_description/meshes/leg_parallel_plate_v1_4.stl" scale="0.001 0.001 0.001"/>
-    </geometry>
-    <material name="silver"/>
-  </visual>
-  <collision>
-    <origin rpy="0 0 0" xyz="0.029063 0.026392 -0.010991"/>
-    <geometry>
-      <mesh filename="package://quadruped_urdf_description/meshes/leg_parallel_plate_v1_4.stl" scale="0.001 0.001 0.001"/>
     </geometry>
   </collision>
