Commit message: commit modified urdf
Former-commit-id: bfb98193ba9d7d67de0ce0a63cfa1e1891298002

File: src/simulations/ws/src/quadruped/quadruped_description/urdf/quadruped.xacro (robot description, xacro)
@@ -6,5 +6,5 @@
 <link name="base_link">
   <inertial>
-    <origin rpy="0 0 0" xyz="8.990840418494208e-07 0.0015934088628400953 -3.844423505811462e-06"/>
+    <origin rpy="0 0 0" xyz="1.129613868000441e-06 0.0015931744186381052 -3.7860729041196138e-06"/>
     <mass value="0.03172042156458545"/>
     <inertia ixx="4.9e-05" ixy="0.0" ixz="-0.0" iyy="4.9e-05" iyz="-0.0" izz="9.8e-05"/>
@@ -26,10 +26,10 @@
 <link name="body_spacer_v1_1">
   <inertial>
-    <origin rpy="0 0 0" xyz="-6.81883996429006e-10 -1.490891317831866e-07 0.0019124056524901113"/>
+    <origin rpy="0 0 0" xyz="3.202473670876637e-07 -3.880843210402052e-07 0.0019124815655197271"/>
     <mass value="0.003797653049825268"/>
     <inertia ixx="0.0" ixy="0.0" ixz="-0.0" iyy="1e-06" iyz="0.0" izz="1e-06"/>
   </inertial>
   <visual>
-    <origin rpy="0 0 0" xyz="0.0 -0.044629 -0.00924"/>
+    <origin rpy="0 0 0" xyz="-0.0 -0.044629 -0.00924"/>
     <geometry>
       <mesh filename="package://quadruped_description/meshes/body_spacer_v1_1.stl" scale="0.001 0.001 0.001"/>
@@ -38,5 +38,5 @@
   </visual>
   <collision>
-    <origin rpy="0 0 0" xyz="0.0 -0.044629 -0.00924"/>
+    <origin rpy="0 0 0" xyz="-0.0 -0.044629 -0.00924"/>
     <geometry>
       <mesh filename="package://quadruped_description/meshes/body_spacer_v1_1.stl" scale="0.001 0.001 0.001"/>
@@ -46,10 +46,10 @@
 <link name="body_spacer_v1_2">
   <inertial>
-    <origin rpy="0 0 0" xyz="-1.2978154060811503e-08 3.50910869161003e-07 0.0019124056524900852"/>
+    <origin rpy="0 0 0" xyz="1.1806497426878e-07 1.119159236465106e-07 0.001912446443342217"/>
     <mass value="0.003797653049825268"/>
     <inertia ixx="0.0" ixy="0.0" ixz="-0.0" iyy="1e-06" iyz="0.0" izz="1e-06"/>
   </inertial>
   <visual>
-    <origin rpy="0 0 0" xyz="0.0 0.041434 -0.00924"/>
+    <origin rpy="0 0 0" xyz="-0.0 0.041434 -0.00924"/>
     <geometry>
       <mesh filename="package://quadruped_description/meshes/body_spacer_v1_2.stl" scale="0.001 0.001 0.001"/>
@@ -58,5 +58,5 @@
   </visual>
   <collision>
-    <origin rpy="0 0 0" xyz="0.0 0.041434 -0.00924"/>
+    <origin rpy="0 0 0" xyz="-0.0 0.041434 -0.00924"/>
     <geometry>
       <mesh filename="package://quadruped_description/meshes/body_spacer_v1_2.stl" scale="0.001 0.001 0.001"/>
@@ -66,10 +66,10 @@
 <link name="body_spacer_v1_3">
   <inertial>
-    <origin rpy="0 0 0" xyz="2.4316998048501404e-07 -4.052372663944457e-07 0.001912405652490094"/>
+    <origin rpy="0 0 0" xyz="4.691560483022217e-07 2.6082459757791054e-07 0.0019124815655201678"/>
     <mass value="0.003797653049825268"/>
-    <inertia ixx="1e-06" ixy="-0.0" ixz="-0.0" iyy="0.0" iyz="0.0" izz="1e-06"/>
-  </inertial>
-  <visual>
-    <origin rpy="0 0 0" xyz="-0.043031 -0.001598 -0.00924"/>
+    <inertia ixx="1e-06" ixy="-0.0" ixz="0.0" iyy="0.0" iyz="-0.0" izz="1e-06"/>
+  </inertial>
+  <visual>
+    <origin rpy="0 0 0" xyz="-0.043031 -0.001597 -0.00924"/>
     <geometry>
       <mesh filename="package://quadruped_description/meshes/body_spacer_v1_3.stl" scale="0.001 0.001 0.001"/>
@@ -78,5 +78,5 @@
   </visual>
   <collision>
-    <origin rpy="0 0 0" xyz="-0.043031 -0.001598 -0.00924"/>
+    <origin rpy="0 0 0" xyz="-0.043031 -0.001597 -0.00924"/>
     <geometry>
       <mesh filename="package://quadruped_description/meshes/body_spacer_v1_3.stl" scale="0.001 0.001 0.001"/>
@@ -86,10 +86,10 @@
 <link name="body_spacer_v1_4">
   <inertial>
-    <origin rpy="0 0 0" xyz="-2.5683001855791865e-07 -3.929409962410979e-07 0.0019124056524901026"/>
+    <origin rpy="0 0 0" xyz="-3.084370694267369e-08 4.6300700498060586e-07 0.0019124464433417695"/>
     <mass value="0.003797653049825268"/>
-    <inertia ixx="1e-06" ixy="-0.0" ixz="0.0" iyy="0.0" iyz="0.0" izz="1e-06"/>
-  </inertial>
-  <visual>
-    <origin rpy="0 0 0" xyz="0.043031 -0.001598 -0.00924"/>
+    <inertia ixx="1e-06" ixy="-0.0" ixz="0.0" iyy="0.0" iyz="-0.0" izz="1e-06"/>
+  </inertial>
+  <visual>
+    <origin rpy="0 0 0" xyz="0.043031 -0.001597 -0.00924"/>
     <geometry>
       <mesh filename="package://quadruped_description/meshes/body_spacer_v1_4.stl" scale="0.001 0.001 0.001"/>
@@ -98,5 +98,5 @@
   </visual>
   <collision>
-    <origin rpy="0 0 0" xyz="0.043031 -0.001598 -0.00924"/>
+    <origin rpy="0 0 0" xyz="0.043031 -0.001597 -0.00924"/>
     <geometry>
       <mesh filename="package://quadruped_description/meshes/body_spacer_v1_4.stl" scale="0.001 0.001 0.001"/>
@@ -106,10 +106,10 @@
 <link name="body_top_plate_v1_1">
   <inertial>
-    <origin rpy="0 0 0" xyz="-6.224116379125583e-06 -7.854114594208969e-07 0.0015936555764941435"/>
+    <origin rpy="0 0 0" xyz="-7.002672895530318e-06 -1.0289236095511762e-06 0.0015937139236976983"/>
     <mass value="0.04667238799634045"/>
     <inertia ixx="4.7e-05" ixy="-0.0" ixz="-0.0" iyy="4.5e-05" iyz="-0.0" izz="9.2e-05"/>
   </inertial>
   <visual>
-    <origin rpy="0 0 0" xyz="1e-05 -0.001603 -0.020715"/>
+    <origin rpy="0 0 0" xyz="9e-06 -0.001603 -0.020715"/>
     <geometry>
       <mesh filename="package://quadruped_description/meshes/body_top_plate_v1_1.stl" scale="0.001 0.001 0.001"/>
@@ -118,5 +118,5 @@
   </visual>
   <collision>
-    <origin rpy="0 0 0" xyz="1e-05 -0.001603 -0.020715"/>
+    <origin rpy="0 0 0" xyz="9e-06 -0.001603 -0.020715"/>
     <geometry>
       <mesh filename="package://quadruped_description/meshes/body_top_plate_v1_1.stl" scale="0.001 0.001 0.001"/>
@@ -126,10 +126,10 @@
 <link name="servo_motor_v1_1">
   <inertial>
-    <origin rpy="0 0 0" xyz="0.0034452692547771585 0.0034447558543224954 -0.017291510897469286"/>
+    <origin rpy="0 0 0" xyz="0.003444398764857401 0.0034446055389786637 -0.01729148679276793"/>
     <mass value="0.011377011376072494"/>
     <inertia ixx="1e-06" ixy="-0.0" ixz="0.0" iyy="1e-06" iyz="0.0" izz="1e-06"/>
   </inertial>
   <visual>
-    <origin rpy="0 0 0" xyz="0.045406 0.043805 -0.038004"/>
+    <origin rpy="0 0 0" xyz="0.045405 0.043805 -0.038004"/>
     <geometry>
       <mesh filename="package://quadruped_description/meshes/servo_motor_v1_1.stl" scale="0.001 0.001 0.001"/>
@@ -138,5 +138,5 @@
   </visual>
   <collision>
-    <origin rpy="0 0 0" xyz="0.045406 0.043805 -0.038004"/>
+    <origin rpy="0 0 0" xyz="0.045405 0.043805 -0.038004"/>
     <geometry>
       <mesh filename="package://quadruped_description/meshes/servo_motor_v1_1.stl" scale="0.001 0.001 0.001"/>
@@ -146,10 +146,10 @@
 <link name="servo_motor_v1_2">
   <inertial>
-    <origin rpy="0 0 0" xyz="0.0034452810470038536 -0.0034447141797240566 -0.01729151089746924"/>
+    <origin rpy="0 0 0" xyz="0.0034445954414215815 -0.0034448644953048377 -0.01729145259574283"/>
     <mass value="0.011377011376072494"/>
     <inertia ixx="1e-06" ixy="0.0" ixz="0.0" iyy="1e-06" iyz="-0.0" izz="1e-06"/>
   </inertial>
   <visual>
-    <origin rpy="0 0 0" xyz="0.045406 -0.04688 -0.038004"/>
+    <origin rpy="0 0 0" xyz="0.045405 -0.04688 -0.038004"/>
     <geometry>
       <mesh filename="package://quadruped_description/meshes/servo_motor_v1_2.stl" scale="0.001 0.001 0.001"/>
@@ -158,5 +158,5 @@
   </visual>
   <collision>
-    <origin rpy="0 0 0" xyz="0.045406 -0.04688 -0.038004"/>
+    <origin rpy="0 0 0" xyz="0.045405 -0.04688 -0.038004"/>
     <geometry>
       <mesh filename="package://quadruped_description/meshes/servo_motor_v1_2.stl" scale="0.001 0.001 0.001"/>
@@ -166,5 +166,5 @@
 <link name="servo_motor_v1_3">
   <inertial>
-    <origin rpy="0 0 0" xyz="-0.0034453077511524474 -0.003444708780636907 -0.01729151089746929"/>
+    <origin rpy="0 0 0" xyz="-0.0034449930855500674 -0.0034450442583107213 -0.017291418297141075"/>
     <mass value="0.011377011376072494"/>
     <inertia ixx="1e-06" ixy="-0.0" ixz="-0.0" iyy="1e-06" iyz="-0.0" izz="1e-06"/>
@@ -186,5 +186,5 @@
 <link name="servo_motor_v1_4">
   <inertial>
-    <origin rpy="0 0 0" xyz="-0.0034453195613619245 0.0034448987921656196 -0.017291510897469282"/>
+    <origin rpy="0 0 0" xyz="-0.0034451900577967196 0.0034445633147291155 -0.017291452545530724"/>
     <mass value="0.011377011376072494"/>
     <inertia ixx="1e-06" ixy="0.0" ixz="-0.0" iyy="1e-06" iyz="0.0" izz="1e-06"/>
@@ -206,49 +206,49 @@
 <link name="leg_servo_retainer_v1_1">
   <inertial>
-    <origin rpy="0 0 0" xyz="-0.007975130604850701 -0.007974365433883905 -3.444235058339129e-07"/>
-    <mass value="0.002255974797814701"/>
-    <inertia ixx="0.0" ixy="-0.0" ixz="0.0" iyy="0.0" iyz="0.0" izz="0.0"/>
-  </inertial>
-  <visual>
-    <origin rpy="0 0 0" xyz="0.033325 0.031724 -0.028684"/>
-    <geometry>
-      <mesh filename="package://quadruped_description/meshes/leg_servo_retainer_v1_1.stl" scale="0.001 0.001 0.001"/>
-    </geometry>
-    <material name="silver"/>
-  </visual>
-  <collision>
-    <origin rpy="0 0 0" xyz="0.033325 0.031724 -0.028684"/>
-    <geometry>
-      <mesh filename="package://quadruped_description/meshes/leg_servo_retainer_v1_1.stl" scale="0.001 0.001 0.001"/>
-    </geometry>
-  </collision>
-</link>
-<link name="leg_servo_retainer_v1_2">
-  <inertial>
-    <origin rpy="0 0 0" xyz="-0.007973840241202512 0.007975685679903782 -3.44423505795749e-07"/>
-    <mass value="0.002255974797814701"/>
-    <inertia ixx="0.0" ixy="0.0" ixz="0.0" iyy="0.0" iyz="-0.0" izz="0.0"/>
-  </inertial>
-  <visual>
-    <origin rpy="0 0 0" xyz="0.033325 -0.034799 -0.028684"/>
-    <geometry>
-      <mesh filename="package://quadruped_description/meshes/leg_servo_retainer_v1_2.stl" scale="0.001 0.001 0.001"/>
-    </geometry>
-    <material name="silver"/>
-  </visual>
-  <collision>
-    <origin rpy="0 0 0" xyz="0.033325 -0.034799 -0.028684"/>
-    <geometry>
-      <mesh filename="package://quadruped_description/meshes/leg_servo_retainer_v1_2.stl" scale="0.001 0.001 0.001"/>
-    </geometry>
-  </collision>
-</link>
-<link name="leg_servo_retainer_v1_3">
-  <inertial>
-    <origin rpy="0 0 0" xyz="0.007975092108475412 0.007974412507569487 -3.44423505826974e-07"/>
+    <origin rpy="0 0 0" xyz="-0.007976002887467012 -0.007974520459792966 -3.1977910110517205e-07"/>
     <mass value="0.002255974797814701"/>
     <inertia ixx="0.0" ixy="-0.0" ixz="-0.0" iyy="0.0" iyz="-0.0" izz="0.0"/>
   </inertial>
   <visual>
+    <origin rpy="0 0 0" xyz="0.033324 0.031724 -0.028684"/>
+    <geometry>
+      <mesh filename="package://quadruped_description/meshes/leg_servo_retainer_v1_1.stl" scale="0.001 0.001 0.001"/>
+    </geometry>
+    <material name="silver"/>
+  </visual>
+  <collision>
+    <origin rpy="0 0 0" xyz="0.033324 0.031724 -0.028684"/>
+    <geometry>
+      <mesh filename="package://quadruped_description/meshes/leg_servo_retainer_v1_1.stl" scale="0.001 0.001 0.001"/>
+    </geometry>
+  </collision>
+</link>
+<link name="leg_servo_retainer_v1_2">
+  <inertial>
+    <origin rpy="0 0 0" xyz="-0.00797453055736528 0.007975530650940081 -2.8612125883495376e-07"/>
+    <mass value="0.002255974797814701"/>
+    <inertia ixx="0.0" ixy="0.0" ixz="-0.0" iyy="0.0" iyz="-0.0" izz="0.0"/>
+  </inertial>
+  <visual>
+    <origin rpy="0 0 0" xyz="0.033324 -0.034799 -0.028684"/>
+    <geometry>
+      <mesh filename="package://quadruped_description/meshes/leg_servo_retainer_v1_2.stl" scale="0.001 0.001 0.001"/>
+    </geometry>
+    <material name="silver"/>
+  </visual>
+  <collision>
+    <origin rpy="0 0 0" xyz="0.033324 -0.034799 -0.028684"/>
+    <geometry>
+      <mesh filename="package://quadruped_description/meshes/leg_servo_retainer_v1_2.stl" scale="0.001 0.001 0.001"/>
+    </geometry>
+  </collision>
+</link>
+<link name="leg_servo_retainer_v1_3">
+  <inertial>
+    <origin rpy="0 0 0" xyz="0.007975402060679655 0.007974075234396874 -2.5236288365981796e-07"/>
+    <mass value="0.002255974797814701"/>
+    <inertia ixx="0.0" ixy="-0.0" ixz="-0.0" iyy="0.0" iyz="-0.0" izz="0.0"/>
+  </inertial>
+  <visual>
     <origin rpy="0 0 0" xyz="-0.033325 -0.034922 -0.028684"/>
     <geometry>
@@ -266,7 +266,7 @@
 <link name="leg_servo_retainer_v1_4">
   <inertial>
-    <origin rpy="0 0 0" xyz="0.007973801726844462 -0.00797550106746222 -3.4442350581656567e-07"/>
+    <origin rpy="0 0 0" xyz="0.007973929434895409 -0.007975838337579831 -2.860720904780678e-07"/>
     <mass value="0.002255974797814701"/>
-    <inertia ixx="0.0" ixy="0.0" ixz="0.0" iyy="0.0" iyz="0.0" izz="0.0"/>
+    <inertia ixx="0.0" ixy="0.0" ixz="-0.0" iyy="0.0" iyz="-0.0" izz="0.0"/>
   </inertial>
   <visual>
@@ -286,10 +286,10 @@
 <link name="leg_top_pivot_plate_v1_1">
   <inertial>
-    <origin rpy="0 0 0" xyz="-0.010648487401591071 -0.010577625981699847 -0.0015938444235058594"/>
+    <origin rpy="0 0 0" xyz="-0.010649403620247293 -0.01057774316660038 -0.0015938317930266552"/>
     <mass value="0.003959817737688224"/>
-    <inertia ixx="0.0" ixy="-0.0" ixz="-0.0" iyy="0.0" iyz="0.0" izz="1e-06"/>
-  </inertial>
-  <visual>
-    <origin rpy="0 0 0" xyz="0.045406 0.043805 -0.038004"/>
+    <inertia ixx="0.0" ixy="-0.0" ixz="-0.0" iyy="0.0" iyz="-0.0" izz="1e-06"/>
+  </inertial>
+  <visual>
+    <origin rpy="0 0 0" xyz="0.045405 0.043805 -0.038004"/>
     <geometry>
       <mesh filename="package://quadruped_description/meshes/leg_top_pivot_plate_v1_1.stl" scale="0.001 0.001 0.001"/>
@@ -298,5 +298,5 @@
   </visual>
   <collision>
-    <origin rpy="0 0 0" xyz="0.045406 0.043805 -0.038004"/>
+    <origin rpy="0 0 0" xyz="0.045405 0.043805 -0.038004"/>
     <geometry>
       <mesh filename="package://quadruped_description/meshes/leg_top_pivot_plate_v1_1.stl" scale="0.001 0.001 0.001"/>
@@ -306,10 +306,10 @@
 <link name="leg_top_pivot_plate_v1_2">
   <inertial>
-    <origin rpy="0 0 0" xyz="-0.010577098036419472 0.010649045210793372 -0.00159384442350579"/>
+    <origin rpy="0 0 0" xyz="-0.010780741103034508 0.01044338061290618 -0.001593786259371191"/>
     <mass value="0.003959817737688224"/>
-    <inertia ixx="0.0" ixy="0.0" ixz="0.0" iyy="0.0" iyz="-0.0" izz="1e-06"/>
-  </inertial>
-  <visual>
-    <origin rpy="0 0 0" xyz="0.045406 -0.04688 -0.038004"/>
+    <inertia ixx="0.0" ixy="0.0" ixz="-0.0" iyy="0.0" iyz="-0.0" izz="1e-06"/>
+  </inertial>
+  <visual>
+    <origin rpy="0 0 0" xyz="0.045405 -0.04688 -0.038004"/>
     <geometry>
       <mesh filename="package://quadruped_description/meshes/leg_top_pivot_plate_v1_2.stl" scale="0.001 0.001 0.001"/>
@@ -318,5 +318,5 @@
   </visual>
   <collision>
-    <origin rpy="0 0 0" xyz="0.045406 -0.04688 -0.038004"/>
+    <origin rpy="0 0 0" xyz="0.045405 -0.04688 -0.038004"/>
     <geometry>
       <mesh filename="package://quadruped_description/meshes/leg_top_pivot_plate_v1_2.stl" scale="0.001 0.001 0.001"/>
@@ -326,7 +326,7 @@
 <link name="leg_top_pivot_plate_v1_3">
   <inertial>
-    <origin rpy="0 0 0" xyz="0.010648457824426617 0.010577664075983234 -0.0015938444235058247"/>
+    <origin rpy="0 0 0" xyz="0.010648796487000789 0.010577291634899517 -0.0015937403489607385"/>
     <mass value="0.003959817737688224"/>
-    <inertia ixx="0.0" ixy="-0.0" ixz="0.0" iyy="0.0" iyz="-0.0" izz="1e-06"/>
+    <inertia ixx="0.0" ixy="-0.0" ixz="-0.0" iyy="0.0" iyz="-0.0" izz="1e-06"/>
   </inertial>
   <visual>
@@ -346,7 +346,7 @@
 <link name="leg_top_pivot_plate_v1_4">
   <inertial>
-    <origin rpy="0 0 0" xyz="0.01057703172127173 -0.010648888212722349 -0.0015938444235058247"/>
+    <origin rpy="0 0 0" xyz="0.010577145835385597 -0.010649239070285699 -0.0015937861007030985"/>
     <mass value="0.003959817737688224"/>
-    <inertia ixx="0.0" ixy="0.0" ixz="0.0" iyy="0.0" iyz="0.0" izz="1e-06"/>
+    <inertia ixx="0.0" ixy="0.0" ixz="-0.0" iyy="0.0" iyz="-0.0" izz="1e-06"/>
   </inertial>
   <visual>
@@ -366,5 +366,5 @@
 <link name="leg_servo_mount_v1_1">
   <inertial>
-    <origin rpy="0 0 0" xyz="-0.0064271966028663155 -0.006426520024797322 -0.009351515125044188"/>
+    <origin rpy="0 0 0" xyz="-0.00642715874115659 -0.006426603384390814 -0.009351513346211524"/>
     <mass value="0.003626406146686101"/>
     <inertia ixx="1e-06" ixy="-0.0" ixz="0.0" iyy="1e-06" iyz="0.0" izz="0.0"/>
@@ -386,10 +386,10 @@
 <link name="leg_servo_mount_v1_2">
   <inertial>
-    <origin rpy="0 0 0" xyz="-0.006426989840584776 0.0064267590464385516 -0.00935151512504408"/>
+    <origin rpy="0 0 0" xyz="-0.006548982610039278 0.0063024928591933205 -0.009351460950992766"/>
     <mass value="0.003626406146686101"/>
     <inertia ixx="1e-06" ixy="0.0" ixz="0.0" iyy="1e-06" iyz="-0.0" izz="0.0"/>
   </inertial>
   <visual>
-    <origin rpy="0 0 0" xyz="0.067485 -0.059764 -0.026529"/>
+    <origin rpy="0 0 0" xyz="0.067729 -0.059336 -0.026529"/>
     <geometry>
       <mesh filename="package://quadruped_description/meshes/leg_servo_mount_v1_2.stl" scale="0.001 0.001 0.001"/>
@@ -398,5 +398,5 @@
   </visual>
   <collision>
-    <origin rpy="0 0 0" xyz="0.067485 -0.059764 -0.026529"/>
+    <origin rpy="0 0 0" xyz="0.067729 -0.059336 -0.026529"/>
     <geometry>
       <mesh filename="package://quadruped_description/meshes/leg_servo_mount_v1_2.stl" scale="0.001 0.001 0.001"/>
@@ -406,10 +406,10 @@
 <link name="leg_servo_mount_v1_3">
   <inertial>
-    <origin rpy="0 0 0" xyz="0.006427182143724279 0.006426550815336579 -0.009351515125044178"/>
+    <origin rpy="0 0 0" xyz="0.00642656730557984 0.006427167550441509 -0.009351400198846106"/>
     <mass value="0.003626406146686101"/>
     <inertia ixx="1e-06" ixy="-0.0" ixz="-0.0" iyy="1e-06" iyz="-0.0" izz="0.0"/>
   </inertial>
   <visual>
-    <origin rpy="0 0 0" xyz="-0.058289 -0.069083 -0.026529"/>
+    <origin rpy="0 0 0" xyz="-0.05829 -0.069082 -0.026529"/>
     <geometry>
       <mesh filename="package://quadruped_description/meshes/leg_servo_mount_v1_3.stl" scale="0.001 0.001 0.001"/>
@@ -418,5 +418,5 @@
   </visual>
   <collision>
-    <origin rpy="0 0 0" xyz="-0.058289 -0.069083 -0.026529"/>
+    <origin rpy="0 0 0" xyz="-0.05829 -0.069082 -0.026529"/>
     <geometry>
       <mesh filename="package://quadruped_description/meshes/leg_servo_mount_v1_3.stl" scale="0.001 0.001 0.001"/>
@@ -426,5 +426,5 @@
 <link name="leg_servo_mount_v1_4">
   <inertial>
-    <origin rpy="0 0 0" xyz="0.006426900912561234 -0.006426648854630061 -0.009351515125044157"/>
+    <origin rpy="0 0 0" xyz="0.006427021750966128 -0.006426994191129902 -0.0093514530202993"/>
     <mass value="0.003626406146686101"/>
     <inertia ixx="1e-06" ixy="0.0" ixz="-0.0" iyy="1e-06" iyz="0.0" izz="0.0"/>
@@ -446,5 +446,5 @@
 <link name="servo_motor_v1_5">
   <inertial>
-    <origin rpy="0 0 0" xyz="0.005636221032410321 -0.0056360238259114265 -0.01221286445355164"/>
+    <origin rpy="0 0 0" xyz="0.005636236407519701 -0.00563611652423214 -0.01221286446387034"/>
     <mass value="0.011377011376072494"/>
     <inertia ixx="1e-06" ixy="0.0" ixz="-0.0" iyy="1e-06" iyz="0.0" izz="1e-06"/>
@@ -466,10 +466,10 @@
 <link name="servo_motor_v1_6">
   <inertial>
-    <origin rpy="0 0 0" xyz="-0.005636494532030675 -0.005636656565279188 -0.012212864453552161"/>
+    <origin rpy="0 0 0" xyz="-0.0055267558784320575 -0.005743927870294624 -0.012212814913568413"/>
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