Commit message: commit modification urdf model
Former-commit-id: 1c760915d958d68c962b3863144a4a68fcccef23

File: src/simulations/ws/src/quadruped/quadruped_description/urdf/quadruped.xacro (robot description, xacro)
@@ -1164,4 +1164,84 @@
   </collision>
 </link>
+<link name="leg_parallel_linkage_v1_1">
+  <inertial>
+    <origin rpy="0 0 0" xyz="-0.007888666974185235 -0.010142013576040165 3.909389618555331e-05"/>
+    <mass value="0.007660744416023881"/>
+    <inertia ixx="0.0" ixy="-0.0" ixz="0.0" iyy="0.0" iyz="0.0" izz="1e-06"/>
+  </inertial>
+  <visual>
+    <origin rpy="0 0 0" xyz="0.073486 0.067901 -0.027613"/>
+    <geometry>
+      <mesh filename="package://quadruped_description/meshes/leg_parallel_linkage_v1_1.stl" scale="0.001 0.001 0.001"/>
+    </geometry>
+    <material name="silver"/>
+  </visual>
+  <collision>
+    <origin rpy="0 0 0" xyz="0.073486 0.067901 -0.027613"/>
+    <geometry>
+      <mesh filename="package://quadruped_description/meshes/leg_parallel_linkage_v1_1.stl" scale="0.001 0.001 0.001"/>
+    </geometry>
+  </collision>
+</link>
+<link name="leg_parallel_linkage_v1_2">
+  <inertial>
+    <origin rpy="0 0 0" xyz="-0.01014253624722418 0.007888263139133309 -3.457620552892171e-07"/>
+    <mass value="0.007660744416023881"/>
+    <inertia ixx="0.0" ixy="0.0" ixz="-0.0" iyy="0.0" iyz="0.0" izz="1e-06"/>
+  </inertial>
+  <visual>
+    <origin rpy="0 0 0" xyz="0.069501 -0.074961 -0.027613"/>
+    <geometry>
+      <mesh filename="package://quadruped_description/meshes/leg_parallel_linkage_v1_2.stl" scale="0.001 0.001 0.001"/>
+    </geometry>
+    <material name="silver"/>
+  </visual>
+  <collision>
+    <origin rpy="0 0 0" xyz="0.069501 -0.074961 -0.027613"/>
+    <geometry>
+      <mesh filename="package://quadruped_description/meshes/leg_parallel_linkage_v1_2.stl" scale="0.001 0.001 0.001"/>
+    </geometry>
+  </collision>
+</link>
+<link name="leg_parallel_linkage_v1_3">
+  <inertial>
+    <origin rpy="0 0 0" xyz="0.00788870492331685 0.010142077319838835 -3.4451109130403945e-07"/>
+    <mass value="0.007660744416023881"/>
+    <inertia ixx="0.0" ixy="-0.0" ixz="-0.0" iyy="0.0" iyz="-0.0" izz="1e-06"/>
+  </inertial>
+  <visual>
+    <origin rpy="0 0 0" xyz="-0.073486 -0.071099 -0.027613"/>
+    <geometry>
+      <mesh filename="package://quadruped_description/meshes/leg_parallel_linkage_v1_3.stl" scale="0.001 0.001 0.001"/>
+    </geometry>
+    <material name="silver"/>
+  </visual>
+  <collision>
+    <origin rpy="0 0 0" xyz="-0.073486 -0.071099 -0.027613"/>
+    <geometry>
+      <mesh filename="package://quadruped_description/meshes/leg_parallel_linkage_v1_3.stl" scale="0.001 0.001 0.001"/>
+    </geometry>
+  </collision>
+</link>
+<link name="leg_parallel_linkage_v1_4">
+  <inertial>
+    <origin rpy="0 0 0" xyz="0.010142332218490771 -0.007889119814119994 4.663672841382499e-05"/>
+    <mass value="0.007660744416023881"/>
+    <inertia ixx="0.0" ixy="0.0" ixz="-0.0" iyy="0.0" iyz="0.0" izz="1e-06"/>
+  </inertial>
+  <visual>
+    <origin rpy="0 0 0" xyz="-0.069501 0.071888 -0.027613"/>
+    <geometry>
+      <mesh filename="package://quadruped_description/meshes/leg_parallel_linkage_v1_4.stl" scale="0.001 0.001 0.001"/>
+    </geometry>
+    <material name="silver"/>
+  </visual>
+  <collision>
+    <origin rpy="0 0 0" xyz="-0.069501 0.071888 -0.027613"/>
+    <geometry>
+      <mesh filename="package://quadruped_description/meshes/leg_parallel_linkage_v1_4.stl" scale="0.001 0.001 0.001"/>
+    </geometry>
+  </collision>
+</link>
 <joint name="Rigid1" type="fixed">
   <origin rpy="0 0 0" xyz="0.0 0.044629 0.00924"/>
@@ -1485,3 +1565,27 @@
   <axis xyz="0.70711 0.707103 -0.0"/>
 </joint>
+<joint name="Rev74" type="continuous">
+  <origin rpy="0 0 0" xyz="0.000614 -0.000614 0.0"/>
+  <parent link="leg_parallel_plate_v1_1"/>
+  <child link="leg_parallel_linkage_v1_1"/>
+  <axis xyz="-0.707109 0.707105 -0.0"/>
+</joint>
+<joint name="Rev75" type="continuous">
+  <origin rpy="0 0 0" xyz="-0.000614 -0.000613 0.0"/>
+  <parent link="leg_parallel_plate_v1_2"/>
+  <child link="leg_parallel_linkage_v1_2"/>
+  <axis xyz="0.707105 0.707109 0.0"/>
+</joint>
+<joint name="Rev76" type="continuous">
+  <origin rpy="0 0 0" xyz="-0.000614 0.000614 0.0"/>
+  <parent link="leg_parallel_plate_v1_3"/>
+  <child link="leg_parallel_linkage_v1_3"/>
+  <axis xyz="0.707108 -0.707105 0.0"/>
+</joint>
+<joint name="Rev77" type="continuous">
+  <origin rpy="0 0 0" xyz="0.000614 0.000614 0.0"/>
+  <parent link="leg_parallel_plate_v1_4"/>
+  <child link="leg_parallel_linkage_v1_4"/>
+  <axis xyz="-0.707107 -0.707107 -0.0"/>
+</joint>
 </robot>

Commit message: commit urdf model
Former-commit-id: 7c81551f8318091e0342a93ff48a7c0a469bbf38

File: src/simulations/ws/src/quadruped/quadruped_description/urdf/quadruped.xacro (robot description, xacro)
@@ -6,7 +6,7 @@
 <link name="base_link">
   <inertial>
-    <origin rpy="0 0 0" xyz="9.020183166175012e-07 0.0015934100491627728 -3.844423505806882e-06"/>
-    <mass value="0.03172042156458545"/>
-    <inertia ixx="4.9e-05" ixy="0.0" ixz="-0.0" iyy="4.9e-05" iyz="-0.0" izz="9.8e-05"/>
+    <origin rpy="0 0 0" xyz="9.059146598178436e-07 0.0015934023756066268 -3.844423505793004e-06"/>
+    <mass value="0.1660035395213305"/>
+    <inertia ixx="0.000257" ixy="0.0" ixz="0.0" iyy="0.000257" iyz="-0.0" izz="0.000514"/>
   </inertial>
   <visual>
@@ -26,10 +26,10 @@
 <link name="body_spacer_v1_1">
   <inertial>
-    <origin rpy="0 0 0" xyz="5.025436629208774e-09 -1.479027513101583e-07 0.0019124056524901286"/>
-    <mass value="0.003797653049825268"/>
-    <inertia ixx="0.0" ixy="0.0" ixz="-0.0" iyy="1e-06" iyz="-0.0" izz="1e-06"/>
-  </inertial>
-  <visual>
-    <origin rpy="0 0 0" xyz="-0.0 -0.044629 -0.00924"/>
+    <origin rpy="0 0 0" xyz="2.7755575615628914e-19 3.4442350579921843e-07 0.0019124056524901113"/>
+    <mass value="0.01987438429408557"/>
+    <inertia ixx="1e-06" ixy="-0.0" ixz="0.0" iyy="4e-06" iyz="0.0" izz="3e-06"/>
+  </inertial>
+  <visual>
+    <origin rpy="0 0 0" xyz="-0.0 0.041434 -0.00924"/>
     <geometry>
       <mesh filename="package://quadruped_description/meshes/body_spacer_v1_1.stl" scale="0.001 0.001 0.001"/>
@@ -38,5 +38,5 @@
   </visual>
   <collision>
-    <origin rpy="0 0 0" xyz="-0.0 -0.044629 -0.00924"/>
+    <origin rpy="0 0 0" xyz="-0.0 0.041434 -0.00924"/>
     <geometry>
       <mesh filename="package://quadruped_description/meshes/body_spacer_v1_1.stl" scale="0.001 0.001 0.001"/>
@@ -46,10 +46,10 @@
 <link name="body_spacer_v1_2">
   <inertial>
-    <origin rpy="0 0 0" xyz="-1.2816384902097095e-08 3.520972508067044e-07 0.0019124056524900766"/>
-    <mass value="0.003797653049825268"/>
-    <inertia ixx="0.0" ixy="0.0" ixz="-0.0" iyy="1e-06" iyz="-0.0" izz="1e-06"/>
-  </inertial>
-  <visual>
-    <origin rpy="0 0 0" xyz="0.0 0.041434 -0.00924"/>
+    <origin rpy="0 0 0" xyz="-6.938893903907229e-19 -1.555764942082205e-07 0.001912405652490139"/>
+    <mass value="0.01987438429408557"/>
+    <inertia ixx="1e-06" ixy="-0.0" ixz="0.0" iyy="4e-06" iyz="0.0" izz="3e-06"/>
+  </inertial>
+  <visual>
+    <origin rpy="0 0 0" xyz="0.0 -0.044629 -0.00924"/>
     <geometry>
       <mesh filename="package://quadruped_description/meshes/body_spacer_v1_2.stl" scale="0.001 0.001 0.001"/>
@@ -58,5 +58,5 @@
   </visual>
   <collision>
-    <origin rpy="0 0 0" xyz="0.0 0.041434 -0.00924"/>
+    <origin rpy="0 0 0" xyz="0.0 -0.044629 -0.00924"/>
     <geometry>
       <mesh filename="package://quadruped_description/meshes/body_spacer_v1_2.stl" scale="0.001 0.001 0.001"/>
@@ -66,12 +66,32 @@
 <link name="body_spacer_v1_3">
   <inertial>
-    <origin rpy="0 0 0" xyz="2.4610452482171086e-07 -4.0682366106502103e-07 0.0019124056524901026"/>
-    <mass value="0.003797653049825268"/>
-    <inertia ixx="1e-06" ixy="-0.0" ixz="0.0" iyy="0.0" iyz="0.0" izz="1e-06"/>
+    <origin rpy="0 0 0" xyz="-2.4999999999331113e-07 -4.0557649421128945e-07 0.0019124056524901182"/>
+    <mass value="0.01987438429408557"/>
+    <inertia ixx="4e-06" ixy="0.0" ixz="0.0" iyy="1e-06" iyz="-0.0" izz="3e-06"/>
+  </inertial>
+  <visual>
+    <origin rpy="0 0 0" xyz="0.043031 -0.001598 -0.00924"/>
+    <geometry>
+      <mesh filename="package://quadruped_description/meshes/body_spacer_v1_3.stl" scale="0.001 0.001 0.001"/>
+    </geometry>
+    <material name="silver"/>
+  </visual>
+  <collision>
+    <origin rpy="0 0 0" xyz="0.043031 -0.001598 -0.00924"/>
+    <geometry>
+      <mesh filename="package://quadruped_description/meshes/body_spacer_v1_3.stl" scale="0.001 0.001 0.001"/>
+    </geometry>
+  </collision>
+</link>
+<link name="body_spacer_v1_4">
+  <inertial>
+    <origin rpy="0 0 0" xyz="2.4999999999331113e-07 -4.0557649421020525e-07 0.0019124056524901182"/>
+    <mass value="0.01987438429408557"/>
+    <inertia ixx="4e-06" ixy="0.0" ixz="0.0" iyy="1e-06" iyz="-0.0" izz="3e-06"/>
   </inertial>
   <visual>
     <origin rpy="0 0 0" xyz="-0.043031 -0.001598 -0.00924"/>
     <geometry>
-      <mesh filename="package://quadruped_description/meshes/body_spacer_v1_3.stl" scale="0.001 0.001 0.001"/>
+      <mesh filename="package://quadruped_description/meshes/body_spacer_v1_4.stl" scale="0.001 0.001 0.001"/>
     </geometry>
     <material name="silver"/>
@@ -80,36 +100,16 @@
     <origin rpy="0 0 0" xyz="-0.043031 -0.001598 -0.00924"/>
     <geometry>
-      <mesh filename="package://quadruped_description/meshes/body_spacer_v1_3.stl" scale="0.001 0.001 0.001"/>
-    </geometry>
-  </collision>
-</link>
-<link name="body_spacer_v1_4">
-  <inertial>
-    <origin rpy="0 0 0" xyz="-2.538954731109988e-07 -3.8898183947152533e-07 0.0019124056524901026"/>
-    <mass value="0.003797653049825268"/>
-    <inertia ixx="1e-06" ixy="-0.0" ixz="0.0" iyy="0.0" iyz="0.0" izz="1e-06"/>
-  </inertial>
-  <visual>
-    <origin rpy="0 0 0" xyz="0.043031 -0.001598 -0.00924"/>
-    <geometry>
       <mesh filename="package://quadruped_description/meshes/body_spacer_v1_4.stl" scale="0.001 0.001 0.001"/>
     </geometry>
-    <material name="silver"/>
-  </visual>
-  <collision>
-    <origin rpy="0 0 0" xyz="0.043031 -0.001598 -0.00924"/>
-    <geometry>
-      <mesh filename="package://quadruped_description/meshes/body_spacer_v1_4.stl" scale="0.001 0.001 0.001"/>
-    </geometry>
   </collision>
 </link>
 <link name="body_top_plate_v1_1">
   <inertial>
-    <origin rpy="0 0 0" xyz="-6.221181536960989e-06 -7.842240333725669e-07 0.0015936555764941539"/>
-    <mass value="0.04667238799634045"/>
-    <inertia ixx="4.7e-05" ixy="-0.0" ixz="-0.0" iyy="4.5e-05" iyz="-0.0" izz="9.2e-05"/>
-  </inertial>
-  <visual>
-    <origin rpy="0 0 0" xyz="1e-05 -0.001603 -0.020715"/>
+    <origin rpy="0 0 0" xyz="-6.217287019302714e-06 -7.919011395236646e-07 -0.0015933444235057825"/>
+    <mass value="0.2442521638475155"/>
+    <inertia ixx="0.000246" ixy="-0.0" ixz="0.0" iyy="0.000236" iyz="-0.0" izz="0.000482"/>
+  </inertial>
+  <visual>
+    <origin rpy="0 0 0" xyz="1e-05 -0.001603 -0.023902"/>
     <geometry>
       <mesh filename="package://quadruped_description/meshes/body_top_plate_v1_1.stl" scale="0.001 0.001 0.001"/>
@@ -118,5 +118,5 @@
   </visual>
   <collision>
-    <origin rpy="0 0 0" xyz="1e-05 -0.001603 -0.020715"/>
+    <origin rpy="0 0 0" xyz="1e-05 -0.001603 -0.023902"/>
     <geometry>
       <mesh filename="package://quadruped_description/meshes/body_top_plate_v1_1.stl" scale="0.001 0.001 0.001"/>
@@ -126,6 +126,26 @@
 <link name="servo_motor_v1_1">
   <inertial>
-    <origin rpy="0 0 0" xyz="0.003445269485712804 0.0034447597444987113 -0.017291510897469282"/>
-    <mass value="0.011377011376072494"/>
+    <origin rpy="0 0 0" xyz="-0.0034453069163115357 -0.003444709272821221 -0.01729151089746925"/>
+    <mass value="0.008039754705757893"/>
+    <inertia ixx="1e-06" ixy="-0.0" ixz="-0.0" iyy="1e-06" iyz="-0.0" izz="1e-06"/>
+  </inertial>
+  <visual>
+    <origin rpy="0 0 0" xyz="-0.045406 -0.047003 -0.038004"/>
+    <geometry>
+      <mesh filename="package://quadruped_description/meshes/servo_motor_v1_1.stl" scale="0.001 0.001 0.001"/>
+    </geometry>
+    <material name="silver"/>
+  </visual>
+  <collision>
+    <origin rpy="0 0 0" xyz="-0.045406 -0.047003 -0.038004"/>
+    <geometry>
+      <mesh filename="package://quadruped_description/meshes/servo_motor_v1_1.stl" scale="0.001 0.001 0.001"/>
+    </geometry>
+  </collision>
+</link>
+<link name="servo_motor_v1_2">
+  <inertial>
+    <origin rpy="0 0 0" xyz="0.00344528207956777 0.003444743371777498 -0.01729151089746927"/>
+    <mass value="0.008039754705757893"/>
     <inertia ixx="1e-06" ixy="-0.0" ixz="0.0" iyy="1e-06" iyz="0.0" izz="1e-06"/>
   </inertial>
@@ -133,5 +153,5 @@
     <origin rpy="0 0 0" xyz="0.045406 0.043805 -0.038004"/>
     <geometry>
-      <mesh filename="package://quadruped_description/meshes/servo_motor_v1_1.stl" scale="0.001 0.001 0.001"/>
+      <mesh filename="package://quadruped_description/meshes/servo_motor_v1_2.stl" scale="0.001 0.001 0.001"/>
     </geometry>
     <material name="silver"/>
@@ -140,12 +160,32 @@
     <origin rpy="0 0 0" xyz="0.045406 0.043805 -0.038004"/>
     <geometry>
-      <mesh filename="package://quadruped_description/meshes/servo_motor_v1_1.stl" scale="0.001 0.001 0.001"/>
-    </geometry>
-  </collision>
-</link>
-<link name="servo_motor_v1_2">
-  <inertial>
-    <origin rpy="0 0 0" xyz="0.0034452866774157542 -0.0034447102895489856 -0.01729151089746925"/>
-    <mass value="0.011377011376072494"/>
+      <mesh filename="package://quadruped_description/meshes/servo_motor_v1_2.stl" scale="0.001 0.001 0.001"/>
+    </geometry>
+  </collision>
+</link>
+<link name="servo_motor_v1_3">
+  <inertial>
+    <origin rpy="0 0 0" xyz="-0.003445306736163896 0.0034448982999804242 -0.017291510897469293"/>
+    <mass value="0.008039754705757893"/>
+    <inertia ixx="1e-06" ixy="0.0" ixz="-0.0" iyy="1e-06" iyz="0.0" izz="1e-06"/>
+  </inertial>
+  <visual>
+    <origin rpy="0 0 0" xyz="-0.045406 0.043808 -0.038004"/>
+    <geometry>
+      <mesh filename="package://quadruped_description/meshes/servo_motor_v1_3.stl" scale="0.001 0.001 0.001"/>
+    </geometry>
+    <material name="silver"/>
+  </visual>
+  <collision>
+    <origin rpy="0 0 0" xyz="-0.045406 0.043808 -0.038004"/>
+    <geometry>
+      <mesh filename="package://quadruped_description/meshes/servo_motor_v1_3.stl" scale="0.001 0.001 0.001"/>
+    </geometry>
+  </collision>
+</link>
+<link name="servo_motor_v1_4">
+  <inertial>
+    <origin rpy="0 0 0" xyz="0.003445281899420151 -0.0034447266622682007 -0.01729151089746927"/>
+    <mass value="0.008039754705757893"/>
     <inertia ixx="1e-06" ixy="0.0" ixz="0.0" iyy="1e-06" iyz="-0.0" izz="1e-06"/>
   </inertial>
@@ -153,5 +193,5 @@
     <origin rpy="0 0 0" xyz="0.045406 -0.04688 -0.038004"/>
     <geometry>
-      <mesh filename="package://quadruped_description/meshes/servo_motor_v1_2.stl" scale="0.001 0.001 0.001"/>
+      <mesh filename="package://quadruped_description/meshes/servo_motor_v1_4.stl" scale="0.001 0.001 0.001"/>
     </geometry>
     <material name="silver"/>
@@ -160,312 +200,312 @@
     <origin rpy="0 0 0" xyz="0.045406 -0.04688 -0.038004"/>
     <geometry>
-      <mesh filename="package://quadruped_description/meshes/servo_motor_v1_2.stl" scale="0.001 0.001 0.001"/>
-    </geometry>
-  </collision>
-</link>
-<link name="servo_motor_v1_3">
-  <inertial>
-    <origin rpy="0 0 0" xyz="-0.0034453021128149353 -0.003444710298049422 -0.017291510897469255"/>
-    <mass value="0.011377011376072494"/>
+      <mesh filename="package://quadruped_description/meshes/servo_motor_v1_4.stl" scale="0.001 0.001 0.001"/>
+    </geometry>
+  </collision>
+</link>
+<link name="leg_servo_retainer_v1_1">
+  <inertial>
+    <origin rpy="0 0 0" xyz="0.007924108380789871 0.007923419580222739 -3.444235058061573e-07"/>
+    <mass value="0.011735752466802122"/>
+    <inertia ixx="1e-06" ixy="-0.0" ixz="-0.0" iyy="1e-06" iyz="0.0" izz="2e-06"/>
+  </inertial>
+  <visual>
+    <origin rpy="0 0 0" xyz="-0.033325 -0.034922 -0.028684"/>
+    <geometry>
+      <mesh filename="package://quadruped_description/meshes/leg_servo_retainer_v1_1.stl" scale="0.001 0.001 0.001"/>
+    </geometry>
+    <material name="silver"/>
+  </visual>
+  <collision>
+    <origin rpy="0 0 0" xyz="-0.033325 -0.034922 -0.028684"/>
+    <geometry>
+      <mesh filename="package://quadruped_description/meshes/leg_servo_retainer_v1_1.stl" scale="0.001 0.001 0.001"/>
+    </geometry>
+  </collision>
+</link>
+<link name="leg_servo_retainer_v1_2">
+  <inertial>
+    <origin rpy="0 0 0" xyz="-0.007924133217533623 -0.007923385481266518 -3.4442350583044345e-07"/>
+    <mass value="0.011735752466802122"/>
+    <inertia ixx="1e-06" ixy="-0.0" ixz="-0.0" iyy="1e-06" iyz="-0.0" izz="2e-06"/>
+  </inertial>
+  <visual>
+    <origin rpy="0 0 0" xyz="0.033325 0.031724 -0.028684"/>
+    <geometry>
+      <mesh filename="package://quadruped_description/meshes/leg_servo_retainer_v1_2.stl" scale="0.001 0.001 0.001"/>
+    </geometry>
+    <material name="silver"/>
+  </visual>
+  <collision>
+    <origin rpy="0 0 0" xyz="0.033325 0.031724 -0.028684"/>
+    <geometry>
+      <mesh filename="package://quadruped_description/meshes/leg_servo_retainer_v1_2.stl" scale="0.001 0.001 0.001"/>
+    </geometry>
+  </collision>
+</link>
+<link name="leg_servo_retainer_v1_3">
+  <inertial>
+    <origin rpy="0 0 0" xyz="0.007922822116880057 -0.00792451699712099 -3.444235058547296e-07"/>
+    <mass value="0.011735752466802122"/>
+    <inertia ixx="1e-06" ixy="0.0" ixz="-0.0" iyy="1e-06" iyz="0.0" izz="2e-06"/>
+  </inertial>
+  <visual>
+    <origin rpy="0 0 0" xyz="-0.033325 0.031727 -0.028684"/>
+    <geometry>
+      <mesh filename="package://quadruped_description/meshes/leg_servo_retainer_v1_3.stl" scale="0.001 0.001 0.001"/>
+    </geometry>
+    <material name="silver"/>
+  </visual>
+  <collision>
+    <origin rpy="0 0 0" xyz="-0.033325 0.031727 -0.028684"/>
+    <geometry>
+      <mesh filename="package://quadruped_description/meshes/leg_servo_retainer_v1_3.stl" scale="0.001 0.001 0.001"/>
+    </geometry>
+  </collision>
+</link>
+<link name="leg_servo_retainer_v1_4">
+  <inertial>
+    <origin rpy="0 0 0" xyz="-0.007922846953623781 0.007924688634833164 -3.444235058130962e-07"/>
+    <mass value="0.011735752466802122"/>
+    <inertia ixx="1e-06" ixy="0.0" ixz="0.0" iyy="1e-06" iyz="-0.0" izz="2e-06"/>
+  </inertial>
+  <visual>
+    <origin rpy="0 0 0" xyz="0.033325 -0.034799 -0.028684"/>
+    <geometry>
+      <mesh filename="package://quadruped_description/meshes/leg_servo_retainer_v1_4.stl" scale="0.001 0.001 0.001"/>
+    </geometry>
+    <material name="silver"/>
+  </visual>
+  <collision>
+    <origin rpy="0 0 0" xyz="0.033325 -0.034799 -0.028684"/>
+    <geometry>
+      <mesh filename="package://quadruped_description/meshes/leg_servo_retainer_v1_4.stl" scale="0.001 0.001 0.001"/>
+    </geometry>
+  </collision>
+</link>
+<link name="leg_top_pivot_plate_v1_1">
+  <inertial>
+    <origin rpy="0 0 0" xyz="0.010648424399168688 0.010577698071700989 -0.0015938444235058177"/>
+    <mass value="0.020723046160568363"/>
+    <inertia ixx="2e-06" ixy="-1e-06" ixz="0.0" iyy="2e-06" iyz="0.0" izz="4e-06"/>
+  </inertial>
+  <visual>
+    <origin rpy="0 0 0" xyz="-0.045406 -0.047003 -0.038004"/>
+    <geometry>
+      <mesh filename="package://quadruped_description/meshes/leg_top_pivot_plate_v1_1.stl" scale="0.001 0.001 0.001"/>
+    </geometry>
+    <material name="silver"/>
+  </visual>
+  <collision>
+    <origin rpy="0 0 0" xyz="-0.045406 -0.047003 -0.038004"/>
+    <geometry>
+      <mesh filename="package://quadruped_description/meshes/leg_top_pivot_plate_v1_1.stl" scale="0.001 0.001 0.001"/>
+    </geometry>
+  </collision>
+</link>
+<link name="leg_top_pivot_plate_v1_2">
+  <inertial>
+    <origin rpy="0 0 0" xyz="-0.010648449235912509 -0.010577663972744698 -0.0015938444235058594"/>
+    <mass value="0.020723046160568363"/>
+    <inertia ixx="2e-06" ixy="-1e-06" ixz="0.0" iyy="2e-06" iyz="0.0" izz="4e-06"/>
+  </inertial>
+  <visual>
+    <origin rpy="0 0 0" xyz="0.045406 0.043805 -0.038004"/>
+    <geometry>
+      <mesh filename="package://quadruped_description/meshes/leg_top_pivot_plate_v1_2.stl" scale="0.001 0.001 0.001"/>
+    </geometry>
+    <material name="silver"/>
+  </visual>
+  <collision>
+    <origin rpy="0 0 0" xyz="0.045406 0.043805 -0.038004"/>
+    <geometry>
+      <mesh filename="package://quadruped_description/meshes/leg_top_pivot_plate_v1_2.stl" scale="0.001 0.001 0.001"/>
+    </geometry>
+  </collision>
+</link>
+<link name="leg_top_pivot_plate_v1_3">
+  <inertial>
+    <origin rpy="0 0 0" xyz="0.010577100608358356 -0.010648833015499792 -0.0015938444235058871"/>
+    <mass value="0.020723046160568363"/>
+    <inertia ixx="2e-06" ixy="1e-06" ixz="0.0" iyy="2e-06" iyz="-0.0" izz="4e-06"/>
+  </inertial>
+  <visual>
+    <origin rpy="0 0 0" xyz="-0.045406 0.043808 -0.038004"/>
+    <geometry>
+      <mesh filename="package://quadruped_description/meshes/leg_top_pivot_plate_v1_3.stl" scale="0.001 0.001 0.001"/>
+    </geometry>
+    <material name="silver"/>
+  </visual>
+  <collision>
+    <origin rpy="0 0 0" xyz="-0.045406 0.043808 -0.038004"/>
+    <geometry>
+      <mesh filename="package://quadruped_description/meshes/leg_top_pivot_plate_v1_3.stl" scale="0.001 0.001 0.001"/>
+    </geometry>
+  </collision>
+</link>
+<link name="leg_top_pivot_plate_v1_4">
+  <inertial>
+    <origin rpy="0 0 0" xyz="-0.010577125445102108 0.010649004653212044 -0.0015938444235058385"/>
+    <mass value="0.020723046160568363"/>
+    <inertia ixx="2e-06" ixy="1e-06" ixz="0.0" iyy="2e-06" iyz="0.0" izz="4e-06"/>
+  </inertial>
+  <visual>
+    <origin rpy="0 0 0" xyz="0.045406 -0.04688 -0.038004"/>
+    <geometry>
+      <mesh filename="package://quadruped_description/meshes/leg_top_pivot_plate_v1_4.stl" scale="0.001 0.001 0.001"/>
+    </geometry>
+    <material name="silver"/>
+  </visual>
+  <collision>
+    <origin rpy="0 0 0" xyz="0.045406 -0.04688 -0.038004"/>
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