Commit message: commit urdf y shift above ground
Former-commit-id: 866371983dcc943b0ddb9fe14f1ede537823b740

File: src/simulations/ws/src/quadruped/quadruped_description/urdf/quadruped.xacro (robot description, xacro)
@@ -6,5 +6,5 @@
 <link name="base_link">
   <inertial>
-    <origin rpy="0 0 0" xyz="9.059146598178436e-07 0.0015934023756066268 -3.844423505793004e-06"/>
+    <origin rpy="0 0 0" xyz="9.059146598001685e-07 0.0015934023756066099 0.049996155576494214"/>
     <mass value="0.1660035395213305"/>
     <inertia ixx="0.000257" ixy="0.0" ixz="0.0" iyy="0.000257" iyz="-0.0" izz="0.000514"/>
@@ -26,10 +26,10 @@
 <link name="body_spacer_v1_1">
   <inertial>
-    <origin rpy="0 0 0" xyz="2.7755575615628914e-19 3.4442350579921843e-07 0.0019124056524901113"/>
+    <origin rpy="0 0 0" xyz="-2.3037127760971997e-17 3.4442350579921843e-07 0.0019124056524901095"/>
     <mass value="0.01987438429408557"/>
-    <inertia ixx="1e-06" ixy="-0.0" ixz="0.0" iyy="4e-06" iyz="0.0" izz="3e-06"/>
-  </inertial>
-  <visual>
-    <origin rpy="0 0 0" xyz="-0.0 0.041434 -0.00924"/>
+    <inertia ixx="1e-06" ixy="0.0" ixz="0.0" iyy="4e-06" iyz="0.0" izz="3e-06"/>
+  </inertial>
+  <visual>
+    <origin rpy="0 0 0" xyz="0.0 0.041434 -0.05924"/>
     <geometry>
       <mesh filename="package://quadruped_description/meshes/body_spacer_v1_1.stl" scale="0.001 0.001 0.001"/>
@@ -38,5 +38,5 @@
   </visual>
   <collision>
-    <origin rpy="0 0 0" xyz="-0.0 0.041434 -0.00924"/>
+    <origin rpy="0 0 0" xyz="0.0 0.041434 -0.05924"/>
     <geometry>
       <mesh filename="package://quadruped_description/meshes/body_spacer_v1_1.stl" scale="0.001 0.001 0.001"/>
@@ -46,10 +46,10 @@
 <link name="body_spacer_v1_2">
   <inertial>
-    <origin rpy="0 0 0" xyz="-6.938893903907229e-19 -1.555764942082205e-07 0.001912405652490139"/>
+    <origin rpy="0 0 0" xyz="-1.762479051592436e-17 -1.555764942290372e-07 0.0019124056524901373"/>
     <mass value="0.01987438429408557"/>
-    <inertia ixx="1e-06" ixy="-0.0" ixz="0.0" iyy="4e-06" iyz="0.0" izz="3e-06"/>
-  </inertial>
-  <visual>
-    <origin rpy="0 0 0" xyz="0.0 -0.044629 -0.00924"/>
+    <inertia ixx="1e-06" ixy="0.0" ixz="0.0" iyy="4e-06" iyz="0.0" izz="3e-06"/>
+  </inertial>
+  <visual>
+    <origin rpy="0 0 0" xyz="0.0 -0.044629 -0.05924"/>
     <geometry>
       <mesh filename="package://quadruped_description/meshes/body_spacer_v1_2.stl" scale="0.001 0.001 0.001"/>
@@ -58,5 +58,5 @@
   </visual>
   <collision>
-    <origin rpy="0 0 0" xyz="0.0 -0.044629 -0.00924"/>
+    <origin rpy="0 0 0" xyz="0.0 -0.044629 -0.05924"/>
     <geometry>
       <mesh filename="package://quadruped_description/meshes/body_spacer_v1_2.stl" scale="0.001 0.001 0.001"/>
@@ -66,30 +66,30 @@
 <link name="body_spacer_v1_3">
   <inertial>
-    <origin rpy="0 0 0" xyz="-2.4999999999331113e-07 -4.0557649421128945e-07 0.0019124056524901182"/>
+    <origin rpy="0 0 0" xyz="-2.500000000071889e-07 -4.055764942221315e-07 0.0019124056524901165"/>
+    <mass value="0.01987438429408557"/>
+    <inertia ixx="4e-06" ixy="0.0" ixz="-0.0" iyy="1e-06" iyz="-0.0" izz="3e-06"/>
+  </inertial>
+  <visual>
+    <origin rpy="0 0 0" xyz="0.043031 -0.001598 -0.05924"/>
+    <geometry>
+      <mesh filename="package://quadruped_description/meshes/body_spacer_v1_3.stl" scale="0.001 0.001 0.001"/>
+    </geometry>
+    <material name="silver"/>
+  </visual>
+  <collision>
+    <origin rpy="0 0 0" xyz="0.043031 -0.001598 -0.05924"/>
+    <geometry>
+      <mesh filename="package://quadruped_description/meshes/body_spacer_v1_3.stl" scale="0.001 0.001 0.001"/>
+    </geometry>
+  </collision>
+</link>
+<link name="body_spacer_v1_4">
+  <inertial>
+    <origin rpy="0 0 0" xyz="2.4999999997249445e-07 -4.0557649422690197e-07 0.0019124056524901165"/>
     <mass value="0.01987438429408557"/>
     <inertia ixx="4e-06" ixy="0.0" ixz="0.0" iyy="1e-06" iyz="-0.0" izz="3e-06"/>
   </inertial>
   <visual>
-    <origin rpy="0 0 0" xyz="0.043031 -0.001598 -0.00924"/>
-    <geometry>
-      <mesh filename="package://quadruped_description/meshes/body_spacer_v1_3.stl" scale="0.001 0.001 0.001"/>
-    </geometry>
-    <material name="silver"/>
-  </visual>
-  <collision>
-    <origin rpy="0 0 0" xyz="0.043031 -0.001598 -0.00924"/>
-    <geometry>
-      <mesh filename="package://quadruped_description/meshes/body_spacer_v1_3.stl" scale="0.001 0.001 0.001"/>
-    </geometry>
-  </collision>
-</link>
-<link name="body_spacer_v1_4">
-  <inertial>
-    <origin rpy="0 0 0" xyz="2.4999999999331113e-07 -4.0557649421020525e-07 0.0019124056524901182"/>
-    <mass value="0.01987438429408557"/>
-    <inertia ixx="4e-06" ixy="0.0" ixz="0.0" iyy="1e-06" iyz="-0.0" izz="3e-06"/>
-  </inertial>
-  <visual>
-    <origin rpy="0 0 0" xyz="-0.043031 -0.001598 -0.00924"/>
+    <origin rpy="0 0 0" xyz="-0.043031 -0.001598 -0.05924"/>
     <geometry>
       <mesh filename="package://quadruped_description/meshes/body_spacer_v1_4.stl" scale="0.001 0.001 0.001"/>
@@ -98,5 +98,5 @@
   </visual>
   <collision>
-    <origin rpy="0 0 0" xyz="-0.043031 -0.001598 -0.00924"/>
+    <origin rpy="0 0 0" xyz="-0.043031 -0.001598 -0.05924"/>
     <geometry>
       <mesh filename="package://quadruped_description/meshes/body_spacer_v1_4.stl" scale="0.001 0.001 0.001"/>
@@ -106,10 +106,10 @@
 <link name="body_top_plate_v1_1">
   <inertial>
-    <origin rpy="0 0 0" xyz="-6.217287019302714e-06 -7.919011395236646e-07 -0.0015933444235057825"/>
+    <origin rpy="0 0 0" xyz="-6.217287019304255e-06 -7.919011395336392e-07 -0.0015933444235057687"/>
     <mass value="0.2442521638475155"/>
     <inertia ixx="0.000246" ixy="-0.0" ixz="0.0" iyy="0.000236" iyz="-0.0" izz="0.000482"/>
   </inertial>
   <visual>
-    <origin rpy="0 0 0" xyz="1e-05 -0.001603 -0.023902"/>
+    <origin rpy="0 0 0" xyz="1e-05 -0.001603 -0.073902"/>
     <geometry>
       <mesh filename="package://quadruped_description/meshes/body_top_plate_v1_1.stl" scale="0.001 0.001 0.001"/>
@@ -118,5 +118,5 @@
   </visual>
   <collision>
-    <origin rpy="0 0 0" xyz="1e-05 -0.001603 -0.023902"/>
+    <origin rpy="0 0 0" xyz="1e-05 -0.001603 -0.073902"/>
     <geometry>
       <mesh filename="package://quadruped_description/meshes/body_top_plate_v1_1.stl" scale="0.001 0.001 0.001"/>
@@ -126,10 +126,10 @@
 <link name="servo_motor_v1_1">
   <inertial>
-    <origin rpy="0 0 0" xyz="-0.0034453069163115357 -0.003444709272821221 -0.01729151089746925"/>
+    <origin rpy="0 0 0" xyz="-0.0034453069163115357 -0.003444709272821242 -0.017291510897469234"/>
     <mass value="0.008039754705757893"/>
     <inertia ixx="1e-06" ixy="-0.0" ixz="-0.0" iyy="1e-06" iyz="-0.0" izz="1e-06"/>
   </inertial>
   <visual>
-    <origin rpy="0 0 0" xyz="-0.045406 -0.047003 -0.038004"/>
+    <origin rpy="0 0 0" xyz="-0.045406 -0.047003 -0.088004"/>
     <geometry>
       <mesh filename="package://quadruped_description/meshes/servo_motor_v1_1.stl" scale="0.001 0.001 0.001"/>
@@ -138,5 +138,5 @@
   </visual>
   <collision>
-    <origin rpy="0 0 0" xyz="-0.045406 -0.047003 -0.038004"/>
+    <origin rpy="0 0 0" xyz="-0.045406 -0.047003 -0.088004"/>
     <geometry>
       <mesh filename="package://quadruped_description/meshes/servo_motor_v1_1.stl" scale="0.001 0.001 0.001"/>
@@ -146,10 +146,10 @@
 <link name="servo_motor_v1_2">
   <inertial>
-    <origin rpy="0 0 0" xyz="0.00344528207956777 0.003444743371777498 -0.01729151089746927"/>
+    <origin rpy="0 0 0" xyz="0.00344528207956777 0.00344474337177747 -0.017291510897469248"/>
     <mass value="0.008039754705757893"/>
     <inertia ixx="1e-06" ixy="-0.0" ixz="0.0" iyy="1e-06" iyz="0.0" izz="1e-06"/>
   </inertial>
   <visual>
-    <origin rpy="0 0 0" xyz="0.045406 0.043805 -0.038004"/>
+    <origin rpy="0 0 0" xyz="0.045406 0.043805 -0.088004"/>
     <geometry>
       <mesh filename="package://quadruped_description/meshes/servo_motor_v1_2.stl" scale="0.001 0.001 0.001"/>
@@ -158,5 +158,5 @@
   </visual>
   <collision>
-    <origin rpy="0 0 0" xyz="0.045406 0.043805 -0.038004"/>
+    <origin rpy="0 0 0" xyz="0.045406 0.043805 -0.088004"/>
     <geometry>
       <mesh filename="package://quadruped_description/meshes/servo_motor_v1_2.stl" scale="0.001 0.001 0.001"/>
@@ -166,10 +166,10 @@
 <link name="servo_motor_v1_3">
   <inertial>
-    <origin rpy="0 0 0" xyz="-0.003445306736163896 0.0034448982999804242 -0.017291510897469293"/>
+    <origin rpy="0 0 0" xyz="-0.0034453067361639236 0.0034448982999804242 -0.01729151089746929"/>
     <mass value="0.008039754705757893"/>
     <inertia ixx="1e-06" ixy="0.0" ixz="-0.0" iyy="1e-06" iyz="0.0" izz="1e-06"/>
   </inertial>
   <visual>
-    <origin rpy="0 0 0" xyz="-0.045406 0.043808 -0.038004"/>
+    <origin rpy="0 0 0" xyz="-0.045406 0.043808 -0.088004"/>
     <geometry>
       <mesh filename="package://quadruped_description/meshes/servo_motor_v1_3.stl" scale="0.001 0.001 0.001"/>
@@ -178,5 +178,5 @@
   </visual>
   <collision>
-    <origin rpy="0 0 0" xyz="-0.045406 0.043808 -0.038004"/>
+    <origin rpy="0 0 0" xyz="-0.045406 0.043808 -0.088004"/>
     <geometry>
       <mesh filename="package://quadruped_description/meshes/servo_motor_v1_3.stl" scale="0.001 0.001 0.001"/>
@@ -186,10 +186,10 @@
 <link name="servo_motor_v1_4">
   <inertial>
-    <origin rpy="0 0 0" xyz="0.003445281899420151 -0.0034447266622682007 -0.01729151089746927"/>
+    <origin rpy="0 0 0" xyz="0.003445281899420137 -0.0034447266622682077 -0.017291510897469248"/>
     <mass value="0.008039754705757893"/>
     <inertia ixx="1e-06" ixy="0.0" ixz="0.0" iyy="1e-06" iyz="-0.0" izz="1e-06"/>
   </inertial>
   <visual>
-    <origin rpy="0 0 0" xyz="0.045406 -0.04688 -0.038004"/>
+    <origin rpy="0 0 0" xyz="0.045406 -0.04688 -0.088004"/>
     <geometry>
       <mesh filename="package://quadruped_description/meshes/servo_motor_v1_4.stl" scale="0.001 0.001 0.001"/>
@@ -198,5 +198,5 @@
   </visual>
   <collision>
-    <origin rpy="0 0 0" xyz="0.045406 -0.04688 -0.038004"/>
+    <origin rpy="0 0 0" xyz="0.045406 -0.04688 -0.088004"/>
     <geometry>
       <mesh filename="package://quadruped_description/meshes/servo_motor_v1_4.stl" scale="0.001 0.001 0.001"/>
@@ -206,10 +206,10 @@
 <link name="leg_servo_retainer_v1_1">
   <inertial>
-    <origin rpy="0 0 0" xyz="0.007924108380789871 0.007923419580222739 -3.444235058061573e-07"/>
+    <origin rpy="0 0 0" xyz="0.007924108380789864 0.007923419580222718 -3.4442350579921843e-07"/>
     <mass value="0.011735752466802122"/>
     <inertia ixx="1e-06" ixy="-0.0" ixz="-0.0" iyy="1e-06" iyz="0.0" izz="2e-06"/>
   </inertial>
   <visual>
-    <origin rpy="0 0 0" xyz="-0.033325 -0.034922 -0.028684"/>
+    <origin rpy="0 0 0" xyz="-0.033325 -0.034922 -0.078684"/>
     <geometry>
       <mesh filename="package://quadruped_description/meshes/leg_servo_retainer_v1_1.stl" scale="0.001 0.001 0.001"/>
@@ -218,5 +218,5 @@
   </visual>
   <collision>
-    <origin rpy="0 0 0" xyz="-0.033325 -0.034922 -0.028684"/>
+    <origin rpy="0 0 0" xyz="-0.033325 -0.034922 -0.078684"/>
     <geometry>
       <mesh filename="package://quadruped_description/meshes/leg_servo_retainer_v1_1.stl" scale="0.001 0.001 0.001"/>
@@ -226,10 +226,10 @@
 <link name="leg_servo_retainer_v1_2">
   <inertial>
-    <origin rpy="0 0 0" xyz="-0.007924133217533623 -0.007923385481266518 -3.4442350583044345e-07"/>
+    <origin rpy="0 0 0" xyz="-0.007924133217533623 -0.007923385481266532 -3.444235058408518e-07"/>
     <mass value="0.011735752466802122"/>
-    <inertia ixx="1e-06" ixy="-0.0" ixz="-0.0" iyy="1e-06" iyz="-0.0" izz="2e-06"/>
-  </inertial>
-  <visual>
-    <origin rpy="0 0 0" xyz="0.033325 0.031724 -0.028684"/>
+    <inertia ixx="1e-06" ixy="-0.0" ixz="0.0" iyy="1e-06" iyz="-0.0" izz="2e-06"/>
+  </inertial>
+  <visual>
+    <origin rpy="0 0 0" xyz="0.033325 0.031724 -0.078684"/>
     <geometry>
       <mesh filename="package://quadruped_description/meshes/leg_servo_retainer_v1_2.stl" scale="0.001 0.001 0.001"/>
@@ -238,5 +238,5 @@
   </visual>
   <collision>
-    <origin rpy="0 0 0" xyz="0.033325 0.031724 -0.028684"/>
+    <origin rpy="0 0 0" xyz="0.033325 0.031724 -0.078684"/>
     <geometry>
       <mesh filename="package://quadruped_description/meshes/leg_servo_retainer_v1_2.stl" scale="0.001 0.001 0.001"/>
@@ -246,30 +246,30 @@
 <link name="leg_servo_retainer_v1_3">
   <inertial>
-    <origin rpy="0 0 0" xyz="0.007922822116880057 -0.00792451699712099 -3.444235058547296e-07"/>
-    <mass value="0.011735752466802122"/>
-    <inertia ixx="1e-06" ixy="0.0" ixz="-0.0" iyy="1e-06" iyz="0.0" izz="2e-06"/>
-  </inertial>
-  <visual>
-    <origin rpy="0 0 0" xyz="-0.033325 0.031727 -0.028684"/>
-    <geometry>
-      <mesh filename="package://quadruped_description/meshes/leg_servo_retainer_v1_3.stl" scale="0.001 0.001 0.001"/>
-    </geometry>
-    <material name="silver"/>
-  </visual>
-  <collision>
-    <origin rpy="0 0 0" xyz="-0.033325 0.031727 -0.028684"/>
-    <geometry>
-      <mesh filename="package://quadruped_description/meshes/leg_servo_retainer_v1_3.stl" scale="0.001 0.001 0.001"/>
-    </geometry>
-  </collision>
-</link>
-<link name="leg_servo_retainer_v1_4">
-  <inertial>
-    <origin rpy="0 0 0" xyz="-0.007922846953623781 0.007924688634833164 -3.444235058130962e-07"/>
+    <origin rpy="0 0 0" xyz="0.007922822116880023 -0.00792451699712099 -3.444235058547296e-07"/>
     <mass value="0.011735752466802122"/>
     <inertia ixx="1e-06" ixy="0.0" ixz="0.0" iyy="1e-06" iyz="-0.0" izz="2e-06"/>
   </inertial>
   <visual>
-    <origin rpy="0 0 0" xyz="0.033325 -0.034799 -0.028684"/>
+    <origin rpy="0 0 0" xyz="-0.033325 0.031727 -0.078684"/>
+    <geometry>
+      <mesh filename="package://quadruped_description/meshes/leg_servo_retainer_v1_3.stl" scale="0.001 0.001 0.001"/>
+    </geometry>
+    <material name="silver"/>
+  </visual>
+  <collision>
+    <origin rpy="0 0 0" xyz="-0.033325 0.031727 -0.078684"/>
+    <geometry>
+      <mesh filename="package://quadruped_description/meshes/leg_servo_retainer_v1_3.stl" scale="0.001 0.001 0.001"/>
+    </geometry>
+  </collision>
+</link>
+<link name="leg_servo_retainer_v1_4">
+  <inertial>
+    <origin rpy="0 0 0" xyz="-0.007922846953623795 0.007924688634833157 -3.444235058130962e-07"/>
+    <mass value="0.011735752466802122"/>
+    <inertia ixx="1e-06" ixy="0.0" ixz="0.0" iyy="1e-06" iyz="0.0" izz="2e-06"/>
+  </inertial>
+  <visual>
+    <origin rpy="0 0 0" xyz="0.033325 -0.034799 -0.078684"/>
     <geometry>
       <mesh filename="package://quadruped_description/meshes/leg_servo_retainer_v1_4.stl" scale="0.001 0.001 0.001"/>
@@ -278,5 +278,5 @@
   </visual>
   <collision>
-    <origin rpy="0 0 0" xyz="0.033325 -0.034799 -0.028684"/>
+    <origin rpy="0 0 0" xyz="0.033325 -0.034799 -0.078684"/>
     <geometry>
       <mesh filename="package://quadruped_description/meshes/leg_servo_retainer_v1_4.stl" scale="0.001 0.001 0.001"/>
@@ -286,10 +286,10 @@
 <link name="leg_top_pivot_plate_v1_1">
   <inertial>
-    <origin rpy="0 0 0" xyz="0.010648424399168688 0.010577698071700989 -0.0015938444235058177"/>
+    <origin rpy="0 0 0" xyz="0.010648424399168653 0.010577698071700968 -0.0015938444235058108"/>
     <mass value="0.020723046160568363"/>
-    <inertia ixx="2e-06" ixy="-1e-06" ixz="0.0" iyy="2e-06" iyz="0.0" izz="4e-06"/>
-  </inertial>
-  <visual>
-    <origin rpy="0 0 0" xyz="-0.045406 -0.047003 -0.038004"/>
+    <inertia ixx="2e-06" ixy="-1e-06" ixz="-0.0" iyy="2e-06" iyz="-0.0" izz="4e-06"/>
+  </inertial>
+  <visual>
+    <origin rpy="0 0 0" xyz="-0.045406 -0.047003 -0.088004"/>
     <geometry>
       <mesh filename="package://quadruped_description/meshes/leg_top_pivot_plate_v1_1.stl" scale="0.001 0.001 0.001"/>
@@ -298,5 +298,5 @@
   </visual>
   <collision>
-    <origin rpy="0 0 0" xyz="-0.045406 -0.047003 -0.038004"/>
+    <origin rpy="0 0 0" xyz="-0.045406 -0.047003 -0.088004"/>
     <geometry>
       <mesh filename="package://quadruped_description/meshes/leg_top_pivot_plate_v1_1.stl" scale="0.001 0.001 0.001"/>
@@ -306,10 +306,10 @@
 <link name="leg_top_pivot_plate_v1_2">
   <inertial>
-    <origin rpy="0 0 0" xyz="-0.010648449235912509 -0.010577663972744698 -0.0015938444235058594"/>
+    <origin rpy="0 0 0" xyz="-0.010648449235912537 -0.010577663972744698 -0.0015938444235058524"/>
     <mass value="0.020723046160568363"/>
-    <inertia ixx="2e-06" ixy="-1e-06" ixz="0.0" iyy="2e-06" iyz="0.0" izz="4e-06"/>
-  </inertial>
-  <visual>
-    <origin rpy="0 0 0" xyz="0.045406 0.043805 -0.038004"/>
+    <inertia ixx="2e-06" ixy="-1e-06" ixz="-0.0" iyy="2e-06" iyz="-0.0" izz="4e-06"/>
+  </inertial>
+  <visual>
+    <origin rpy="0 0 0" xyz="0.045406 0.043805 -0.088004"/>
     <geometry>
       <mesh filename="package://quadruped_description/meshes/leg_top_pivot_plate_v1_2.stl" scale="0.001 0.001 0.001"/>
@@ -318,5 +318,5 @@
   </visual>
   <collision>
-    <origin rpy="0 0 0" xyz="0.045406 0.043805 -0.038004"/>
+    <origin rpy="0 0 0" xyz="0.045406 0.043805 -0.088004"/>
     <geometry>
       <mesh filename="package://quadruped_description/meshes/leg_top_pivot_plate_v1_2.stl" scale="0.001 0.001 0.001"/>
@@ -326,30 +326,30 @@
 <link name="leg_top_pivot_plate_v1_3">
   <inertial>
-    <origin rpy="0 0 0" xyz="0.010577100608358356 -0.010648833015499792 -0.0015938444235058871"/>
-    <mass value="0.020723046160568363"/>
-    <inertia ixx="2e-06" ixy="1e-06" ixz="0.0" iyy="2e-06" iyz="-0.0" izz="4e-06"/>
-  </inertial>
-  <visual>
-    <origin rpy="0 0 0" xyz="-0.045406 0.043808 -0.038004"/>
-    <geometry>
-      <mesh filename="package://quadruped_description/meshes/leg_top_pivot_plate_v1_3.stl" scale="0.001 0.001 0.001"/>
-    </geometry>
-    <material name="silver"/>
-  </visual>
-  <collision>
-    <origin rpy="0 0 0" xyz="-0.045406 0.043808 -0.038004"/>
-    <geometry>
-      <mesh filename="package://quadruped_description/meshes/leg_top_pivot_plate_v1_3.stl" scale="0.001 0.001 0.001"/>
-    </geometry>
-  </collision>
-</link>
-<link name="leg_top_pivot_plate_v1_4">
-  <inertial>
-    <origin rpy="0 0 0" xyz="-0.010577125445102108 0.010649004653212044 -0.0015938444235058385"/>
+    <origin rpy="0 0 0" xyz="0.010577100608358335 -0.010648833015499813 -0.001593844423505894"/>
     <mass value="0.020723046160568363"/>
     <inertia ixx="2e-06" ixy="1e-06" ixz="0.0" iyy="2e-06" iyz="0.0" izz="4e-06"/>
   </inertial>
   <visual>
-    <origin rpy="0 0 0" xyz="0.045406 -0.04688 -0.038004"/>
+    <origin rpy="0 0 0" xyz="-0.045406 0.043808 -0.088004"/>
+    <geometry>
+      <mesh filename="package://quadruped_description/meshes/leg_top_pivot_plate_v1_3.stl" scale="0.001 0.001 0.001"/>
+    </geometry>
+    <material name="silver"/>
+  </visual>
+  <collision>
+    <origin rpy="0 0 0" xyz="-0.045406 0.043808 -0.088004"/>
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