Commit message: commit simpler collision model complete till parallel plate, need to compute exact COM positions for parallel plates and standard positioning
Former-commit-id: d56fbda78823d0ef69949e8b56d8e7d767011865

File: src/simulations/ws/src/quadruped_description/urdf/quadruped.urdf (robot description, URDF)
Before this commit: robot quadruped, 46 links, 45 joints
Links:
- link base_link: geometry collision box size=0.113187997 0.113187997 0.003188; visual mesh filename=package://quadruped_description/meshes/base_link.stl scale=0.001 0.001 0.001
- link body_spacer_v11: geometry collision box size=0.03825 0.003188 0.019125; visual mesh filename=package://quadruped_description/meshes/body_spacer_v11.stl scale=0.001 0.001 0.001
- link body_spacer_v12: geometry collision box size=0.03825 0.003188 0.019125; visual mesh filename=package://quadruped_description/meshes/body_spacer_v12.stl scale=0.001 0.001 0.001
- link body_spacer_v13: geometry collision box size=0.003188 0.03825 0.019125; visual mesh filename=package://quadruped_description/meshes/body_spacer_v13.stl scale=0.001 0.001 0.001
- link body_spacer_v14: geometry collision box size=0.003188 0.03825 0.019125; visual mesh filename=package://quadruped_description/meshes/body_spacer_v14.stl scale=0.001 0.001 0.001
- link body_top_plate_v11: geometry collision box size=0.113187997 0.113187997 0.003188; visual mesh filename=package://quadruped_description/meshes/body_top_plate_v11.s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 scale=0.001 0.001 0.001
- link bottom_pivot_plate_v11: geometry collision box size=0.048442 0.02040 0.003188; visual mesh filename=package://quadruped_description/meshes/bottom_pivot_plate_v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 scale=0.001 0.001 0.001
- link bottom_pivot_plate_v12: geometry collision box size=0.048442 0.02040 0.003188; visual mesh filename=package://quadruped_description/meshes/bottom_pivot_plate_v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 scale=0.001 0.001 0.001
- link bottom_pivot_plate_v13: geometry collision box size=0.048442 0.02040 0.003188; visual mesh filename=package://quadruped_description/meshes/bottom_pivot_plate_v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 scale=0.001 0.001 0.001
- link bottom_pivot_plate_v14: geometry collision box size=0.048442 0.02040 0.003188; visual mesh filename=package://quadruped_description/meshes/bottom_pivot_plate_v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 scale=0.001 0.001 0.001
- link leg_parallel_linkage_v11: geometry collision mesh filename=package://quadruped_description/meshes/leg_parallel_linkage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 scale=0.001 0.001 0.001; visual mesh filename=package://quadruped_description/meshes/leg_parallel_linkage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 scale=0.001 0.001 0.001
- link leg_parallel_linkage_v12: geometry collision mesh filename=package://quadruped_description/meshes/leg_parallel_linkage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 scale=0.001 0.001 0.001; visual mesh filename=package://quadruped_description/meshes/leg_parallel_linkage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 scale=0.001 0.001 0.001
- link leg_parallel_linkage_v13: geometry collision mesh filename=package://quadruped_description/meshes/leg_parallel_linkage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 scale=0.001 0.001 0.001; visual mesh filename=package://quadruped_description/meshes/leg_parallel_linkage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 scale=0.001 0.001 0.001
- link leg_parallel_linkage_v14: geometry collision mesh filename=package://quadruped_description/meshes/leg_parallel_linkage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 scale=0.001 0.001 0.001; visual mesh filename=package://quadruped_description/meshes/leg_parallel_linkage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 scale=0.001 0.001 0.001
- link leg_parallel_plate_v11: geometry collision box size=0.024137 0.003188 0.036414; visual mesh filename=package://quadruped_description/meshes/leg_parallel_plate_v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 scale=0.001 0.001 0.001
- link leg_parallel_plate_v12: geometry collision box size=0.024137 0.003188 0.036414; visual mesh filename=package://quadruped_description/meshes/leg_parallel_plate_v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 scale=0.001 0.001 0.001
- link leg_parallel_plate_v13: geometry collision box size=0.024137 0.003188 0.036414; visual mesh filename=package://quadruped_description/meshes/leg_parallel_plate_v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 scale=0.001 0.001 0.001
- link leg_parallel_plate_v14: geometry collision mesh filename=package://quadruped_description/meshes/leg_parallel_plate_v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 scale=0.001 0.001 0.001; visual mesh filename=package://quadruped_description/meshes/leg_parallel_plate_v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 scale=0.001 0.001 0.001
- link leg_rev_v11: geometry collision mesh filename=package://quadruped_description/meshes/leg_rev_v11.stl scale=0.001 0.001 0.001; visual mesh filename=package://quadruped_description/meshes/leg_rev_v11.stl scale=0.001 0.001 0.001
- link leg_rev_v12: geometry collision mesh filename=package://quadruped_description/meshes/leg_rev_v12.stl scale=0.001 0.001 0.001; visual mesh filename=package://quadruped_description/meshes/leg_rev_v12.stl scale=0.001 0.001 0.001
- link leg_rev_v13: geometry collision mesh filename=package://quadruped_description/meshes/leg_rev_v13.stl scale=0.001 0.001 0.001; visual mesh filename=package://quadruped_description/meshes/leg_rev_v13.stl scale=0.001 0.001 0.001
- link leg_rev_v14: geometry collision mesh filename=package://quadruped_description/meshes/leg_rev_v14.stl scale=0.001 0.001 0.001; visual mesh filename=package://quadruped_description/meshes/leg_rev_v14.stl scale=0.001 0.001 0.001
- link leg_servo_arm_v11: geometry collision mesh filename=package://quadruped_description/meshes/leg_servo_arm_v11.stl scale=0.001 0.001 0.001; visual mesh filename=package://quadruped_description/meshes/leg_servo_arm_v11.stl scale=0.001 0.001 0.001
- link leg_servo_arm_v12: geometry collision mesh filename=package://quadruped_description/meshes/leg_servo_arm_v12.stl scale=0.001 0.001 0.001; visual mesh filename=package://quadruped_description/meshes/leg_servo_arm_v12.stl scale=0.001 0.001 0.001
- link leg_servo_arm_v13: geometry collision mesh filename=package://quadruped_description/meshes/leg_servo_arm_v13.stl scale=0.001 0.001 0.001; visual mesh filename=package://quadruped_description/meshes/leg_servo_arm_v13.stl scale=0.001 0.001 0.001
- link leg_servo_arm_v14: geometry collision mesh filename=package://quadruped_description/meshes/leg_servo_arm_v14.stl scale=0.001 0.001 0.001; visual mesh filename=package://quadruped_description/meshes/leg_servo_arm_v14.stl scale=0.001 0.001 0.001
- link leg_servo_mount_v11: geometry collision mesh filename=package://quadruped_description/meshes/leg_servo_mount_v11.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 scale=0.001 0.001 0.001; visual mesh filename=package://quadruped_description/meshes/leg_servo_mount_v11.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 scale=0.001 0.001 0.001
- link leg_servo_mount_v12: geometry collision mesh filename=package://quadruped_description/meshes/leg_servo_mount_v12.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 scale=0.001 0.001 0.001; visual mesh filename=package://quadruped_description/meshes/leg_servo_mount_v12.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 scale=0.001 0.001 0.001
- link leg_servo_mount_v13: geometry collision mesh filename=package://quadruped_description/meshes/leg_servo_mount_v13.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 scale=0.001 0.001 0.001; visual mesh filename=package://quadruped_description/meshes/leg_servo_mount_v13.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 scale=0.001 0.001 0.001
- link leg_servo_mount_v14: geometry collision mesh filename=package://quadruped_description/meshes/leg_servo_mount_v14.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 scale=0.001 0.001 0.001; visual mesh filename=package://quadruped_description/meshes/leg_servo_mount_v14.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 scale=0.001 0.001 0.001
- link leg_servo_retainer_v11: geometry collision mesh filename=package://quadruped_description/meshes/leg_servo_retainer_v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 scale=0.001 0.001 0.001; visual mesh filename=package://quadruped_description/meshes/leg_servo_retainer_v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 scale=0.001 0.001 0.001
- link leg_servo_retainer_v12: geometry collision mesh filename=package://quadruped_description/meshes/leg_servo_retainer_v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 scale=0.001 0.001 0.001; visual mesh filename=package://quadruped_description/meshes/leg_servo_retainer_v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 scale=0.001 0.001 0.001
- link leg_servo_retainer_v13: geometry collision mesh filename=package://quadruped_description/meshes/leg_servo_retainer_v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 scale=0.001 0.001 0.001; visual mesh filename=package://quadruped_description/meshes/leg_servo_retainer_v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 scale=0.001 0.001 0.001
- link leg_servo_retainer_v14: geometry collision mesh filename=package://quadruped_description/meshes/leg_servo_retainer_v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 scale=0.001 0.001 0.001; visual mesh filename=package://quadruped_description/meshes/leg_servo_retainer_v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 scale=0.001 0.001 0.001
- link leg_top_pivot_plate_v11: geometry collision box size=0.048442 0.02040 0.003188; visual mesh filename=package://quadruped_description/meshes/leg_top_pivot_plate_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 scale=0.001 0.001 0.001
- link leg_top_pivot_plate_v12: geometry collision box size=0.048442 0.02040 0.003188; visual mesh filename=package://quadruped_description/meshes/leg_top_pivot_plate_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 scale=0.001 0.001 0.001
- link leg_top_pivot_plate_v13: geometry collision box size=0.048442 0.02040 0.003188; visual mesh filename=package://quadruped_description/meshes/leg_top_pivot_plate_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 scale=0.001 0.001 0.001
- link leg_top_pivot_plate_v14: geometry collision box size=0.048442 0.02040 0.003188; visual mesh filename=package://quadruped_description/meshes/leg_top_pivot_plate_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 scale=0.001 0.001 0.001
- link servo_motor_v11: geometry collision mesh filename=package://quadruped_description/meshes/servo_motor_v11.stl scale=0.001 0.001 0.001; visual mesh filename=package://quadruped_description/meshes/servo_motor_v11.stl scale=0.001 0.001 0.001
- link servo_motor_v12: geometry collision mesh filename=package://quadruped_description/meshes/servo_motor_v12.stl scale=0.001 0.001 0.001; visual mesh filename=package://quadruped_description/meshes/servo_motor_v12.stl scale=0.001 0.001 0.001
- link servo_motor_v13: geometry collision mesh filename=package://quadruped_description/meshes/servo_motor_v13.stl scale=0.001 0.001 0.001; visual mesh filename=package://quadruped_description/meshes/servo_motor_v13.stl scale=0.001 0.001 0.001
- link servo_motor_v14: geometry collision mesh filename=package://quadruped_description/meshes/servo_motor_v14.stl scale=0.001 0.001 0.001; visual mesh filename=package://quadruped_description/meshes/servo_motor_v14.stl scale=0.001 0.001 0.001
- link servo_motor_v15: geometry collision mesh filename=package://quadruped_description/meshes/servo_motor_v15.stl scale=0.001 0.001 0.001; visual mesh filename=package://quadruped_description/meshes/servo_motor_v15.stl scale=0.001 0.001 0.001
- link servo_motor_v16: geometry collision mesh filename=package://quadruped_description/meshes/servo_motor_v16.stl scale=0.001 0.001 0.001; visual mesh filename=package://quadruped_description/meshes/servo_motor_v16.stl scale=0.001 0.001 0.001
- link servo_motor_v17: geometry collision mesh filename=package://quadruped_description/meshes/servo_motor_v17.stl scale=0.001 0.001 0.001; visual mesh filename=package://quadruped_description/meshes/servo_motor_v17.stl scale=0.001 0.001 0.001
- link servo_motor_v18: geometry collision mesh filename=package://quadruped_description/meshes/servo_motor_v18.stl scale=0.001 0.001 0.001; visual mesh filename=package://quadruped_description/meshes/servo_motor_v18.stl scale=0.001 0.001 0.001

Commit message: commit simple collision model
Former-commit-id: 000de39d2e2bc2433d1c5f64349417ea37419c34

File: src/simulations/ws/src/quadruped_description/urdf/quadruped.urdf (robot description, URDF)
Before this commit: robot quadruped, 46 links, 45 joints
Links:
- link leg_parallel_linkage_v11: geometry collision box size=0.003188 0.036657 0.011158; visual mesh filename=package://quadruped_description/meshes/leg_parallel_linkage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 scale=0.001 0.001 0.001
- link leg_parallel_linkage_v12: geometry collision box size=0.003188 0.036657 0.011158; visual mesh filename=package://quadruped_description/meshes/leg_parallel_linkage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 scale=0.001 0.001 0.001
- link leg_parallel_linkage_v13: geometry collision box size=0.003188 0.036657 0.011158; visual mesh filename=package://quadruped_description/meshes/leg_parallel_linkage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 scale=0.001 0.001 0.001
- link leg_parallel_linkage_v14: geometry collision box size=0.003188 0.036657 0.011158; visual mesh filename=package://quadruped_description/meshes/leg_parallel_linkage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 scale=0.001 0.001 0.001
- link leg_parallel_plate_v14: geometry collision box size=0.024137 0.003188 0.036414; visual mesh filename=package://quadruped_description/meshes/leg_parallel_plate_v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 scale=0.001 0.001 0.001
- link leg_rev_v11: geometry collision box size=0.003188 0.001275 0.0961554; visual mesh filename=package://quadruped_description/meshes/leg_rev_v11.stl scale=0.001 0.001 0.001
- link leg_rev_v12: geometry collision box size=0.003188 0.001275 0.0961554; visual mesh filename=package://quadruped_description/meshes/leg_rev_v12.stl scale=0.001 0.001 0.001
- link leg_rev_v13: geometry collision box size=0.003188 0.001275 0.0961554; visual mesh filename=package://quadruped_description/meshes/leg_rev_v13.stl scale=0.001 0.001 0.001
- link leg_rev_v14: geometry collision box size=0.003188 0.001275 0.0961554; visual mesh filename=package://quadruped_description/meshes/leg_rev_v14.stl scale=0.001 0.001 0.001
- link leg_servo_arm_v11: geometry collision box size=0.003188 0.039047 0.015937; visual mesh filename=package://quadruped_description/meshes/leg_servo_arm_v11.stl scale=0.001 0.001 0.001
- link leg_servo_arm_v12: geometry collision box size=0.003188 0.039047 0.015937; visual mesh filename=package://quadruped_description/meshes/leg_servo_arm_v12.stl scale=0.001 0.001 0.001
- link leg_servo_arm_v13: geometry collision box size=0.003188 0.039047 0.015937; visual mesh filename=package://quadruped_description/meshes/leg_servo_arm_v13.stl scale=0.001 0.001 0.001
- link leg_servo_arm_v14: geometry collision box size=0.003188 0.039047 0.015937; visual mesh filename=package://quadruped_description/meshes/leg_servo_arm_v14.stl scale=0.001 0.001 0.001

Commit message: commit COM computation functional setup for reward calculation
Former-commit-id: a0282cf4098230bd45c1107fcb6dd5ee754d06c6

File: src/simulations/ws/src/quadruped_description/urdf/quadruped.urdf (robot description, URDF)
Before this commit: robot quadruped, 46 links, 45 joints
Joints:
- removed joint Rev14
- removed joint Rev15
- removed joint Rev16
- removed joint Rev17
- removed joint Rev26
- removed joint Rev27
- removed joint Rev28
- removed joint Rev29
- added joint Leg1Hip: type continuous, parent servo_motor_v14, child leg_top_pivot_plate_v14, origin xyz=0.0 0.0 0.0 rpy=0 0 0, axis 0.0 -0.0 1.0
- added joint Leg1Knee: type continuous, parent servo_motor_v18, child leg_servo_arm_v14, origin xyz=0.040174 0.036189 -0.018807 rpy=0 0 0, axis 0.707107 0.707107 -0.0
- added joint Leg2Hip: type continuous, parent servo_motor_v13, child leg_top_pivot_plate_v13, origin xyz=0.0 0.0 0.0 rpy=0 0 0, axis 0.0 -0.0 1.0
- added joint Leg2Knee: type continuous, parent servo_motor_v17, child leg_servo_arm_v13, origin xyz=0.03792 0.038443 -0.018807 rpy=0 0 0, axis -0.707107 -0.707107 0.0
- added joint Leg3Hip: type continuous, parent servo_motor_v11, child leg_top_pivot_plate_v11, origin xyz=0.0 0.0 0.0 rpy=0 0 0, axis 0.0 -0.0 1.0
- added joint Leg3Knee: type continuous, parent servo_motor_v15, child leg_servo_arm_v11, origin xyz=0.040174 0.036189 -0.018807 rpy=0 0 0, axis 0.707107 -0.707107 -0.0
- added joint Leg4Hip: type continuous, parent servo_motor_v12, child leg_top_pivot_plate_v12, origin xyz=0.0 0.0 0.0 rpy=0 0 0, axis -0.0 -0.0 1.0
- added joint Leg4Knee: type continuous, parent servo_motor_v16, child leg_servo_arm_v12, origin xyz=0.03792 0.038443 -0.018807 rpy=0 0 0, axis -0.707107 0.707107 0.0

Commit message: commit sync
Former-commit-id: 38a9a0d47fb38b66985a398516c607ac09a5556d

File: src/simulations/ws/src/quadruped_description/urdf/quadruped.urdf (robot description, URDF)
Before this commit: robot quadruped, 46 links, 45 joints
Joints:
- joint Leg1Hip: limit (none) -> lower=-1.5707 upper=1.5707 effort=100 velocity=3; type continuous -> revolute
- joint Leg1Knee: limit (none) -> lower=-1.5707 upper=1.5707 effort=100 velocity=3; type continuous -> revolute
- joint Leg2Hip: limit (none) -> lower=-1.5707 upper=1.5707 effort=100 velocity=3; type continuous -> revolute
- joint Leg2Knee: limit (none) -> lower=-1.5707 upper=1.5707 effort=100 velocity=3; type continuous -> revolute
- joint Leg3Hip: limit (none) -> lower=-1.5707 upper=1.5707 effort=100 velocity=3; type continuous -> revolute
- joint Leg3Knee: limit (none) -> lower=-1.5707 upper=1.5707 effort=100 velocity=3; type continuous -> revolute
- joint Leg4Hip: limit (none) -> lower=-1.5707 upper=1.5707 effort=100 velocity=3; type continuous -> revolute
- joint Leg4Knee: limit (none) -> lower=-1.5707 upper=1.5707 effort=100 velocity=3; type continuous -> revolute
- joint Rev30: limit (none) -> lower=-1.5707 upper=1.5707 effort=100 velocity=3; type continuous -> revolute
- joint Rev31: limit (none) -> lower=-1.5707 upper=1.5707 effort=100 velocity=3; type continuous -> revolute
- joint Rev32: limit (none) -> lower=-1.5707 upper=1.5707 effort=100 velocity=3; type continuous -> revolute
- joint Rev33: limit (none) -> lower=-1.5707 upper=1.5707 effort=100 velocity=3; type continuous -> revolute
- joint Rev34: limit (none) -> lower=-1.5707 upper=1.5707 effort=100 velocity=3; type continuous -> revolute
- joint Rev35: limit (none) -> lower=-1.5707 upper=1.5707 effort=100 velocity=3; type continuous -> revolute
- joint Rev36: limit (none) -> lower=-1.5707 upper=1.5707 effort=100 velocity=3; type continuous -> revolute
- joint Rev37: limit (none) -> lower=-1.5707 upper=1.5707 effort=100 velocity=3; type continuous -> revolute
- joint Rev42: limit (none) -> lower=-1.5707 upper=1.5707 effort=100 velocity=3; type continuous -> revolute
- joint Rev43: limit (none) -> lower=-1.5707 upper=1.5707 effort=100 velocity=3; type continuous -> revolute
- joint Rev44: limit (none) -> lower=-1.5707 upper=1.5707 effort=100 velocity=3; type continuous -> revolute
- joint Rev45: limit (none) -> lower=-1.5707 upper=1.5707 effort=100 velocity=3; type continuous -> revolute
- joint Rev46: limit (none) -> lower=-1.5707 upper=1.5707 effort=100 velocity=3; type continuous -> revolute
- joint Rev47: limit (none) -> lower=-1.5707 upper=1.5707 effort=100 velocity=3; type continuous -> revolute
- joint Rev48: limit (none) -> lower=-1.5707 upper=1.5707 effort=100 velocity=3; type continuous -> revolute
- joint Rev49: limit (none) -> lower=-1.5707 upper=1.5707 effort=100 velocity=3; type continuous -> revolute
