Commit message: commit moveit setup done
Former-commit-id: 64a5300ec7a2883355781e61827d6761f45cafe6

File: src/simulations/ws/src/robot/urdf/quadruped.urdf (robot description, URDF)
Before this commit: robot quadruped, 19 links, 18 joints
Links:
- added link dummy
Joints:
- added joint dummy_joint: type fixed, parent dummy, child dummy_link
